Commit message: Grip service added

File: src/shesnar/urdf/sim_gripper_gz.xacro (robot description, xacro)
@@ -45,4 +45,9 @@
             </geometry>
         </collision>
+        <sensor name='sensor_contact' type='contact'>
+            <contact>
+                <collision>collision</collision>
+            </contact>
+        </sensor>
     </link>
  -->
@@ -55,4 +60,5 @@
         </plugin> -->
     <gazebo>
+<<<<<<< HEAD
         <plugin name="gripper_plugin_gz::DynamicDetachableJoint" filename="libgripper_plugin_gz.so">
             <parent_link>can_gripper_1</parent_link>
@@ -83,4 +89,6 @@
             <grip_link>cylinder1_link</grip_link>
         </plugin>
+=======
+>>>>>>> cbe455e (Grip service added)
         <plugin name="gz::sim::systems::DetachableJoint" filename="gz-sim-detachable-joint-system">
             <parent_link>col_gripper</parent_link>
@@ -89,5 +97,9 @@
             <attach_topic>/model/cylinder11/detachable_joint/attach</attach_topic>
             <detach_topic>/model/cylinder11/detachable_joint/detach</detach_topic>
+<<<<<<< HEAD
         </plugin> -->
+=======
+        </plugin>
+>>>>>>> cbe455e (Grip service added)
         <!-- <plugin filename="gz-sim-touchplugin-system" name="gz::sim::systems::TouchPlugin">
             <target>cylinder11</target>
@@ -108,4 +120,23 @@
         </plugin>
  -->
+<<<<<<< HEAD
+=======
+        <plugin filename="gz-sim-triggered-publisher-system" name="gz::sim::systems::TriggeredPublisher">
+            <input type="gz.msgs.Boolean" topic="/attach_topic">
+            <match>data: true</match>
+            </input>
+            <output type="gz.msgs.Empty" topic="/model/cylinder11/detachable_joint/attach">
+                unused: true
+            </output>
+        </plugin>
+        <plugin filename="gz-sim-triggered-publisher-system" name="gz::sim::systems::TriggeredPublisher">
+            <input type="gz.msgs.Boolean" topic="/detach_topic">
+            <match>data: true</match>
+            </input>
+            <output type="gz.msgs.Empty" topic="/model/cylinder11/detachable_joint/detach">
+                unused: true
+            </output>
+        </plugin>
+>>>>>>> cbe455e (Grip service added)
         <!-- <plugin filename="gz-sim-detachable-joint-system" name="gz::sim::systems::DetachableJoint">
             <parent_link>col_gripper</parent_link>
@@ -128,5 +159,9 @@
             <cmd_max>1000</cmd_max>
             <cmd_min>-1000</cmd_min>
+<<<<<<< HEAD
         </plugin> -->
+=======
+        </plugin>
+>>>>>>> cbe455e (Grip service added)
         <!-- <plugin name="gz::sim::systems::DetachableJoint">
         </plugin> -->

Commit message: Grip service added

File: src/shesnar/urdf/sim_gripper_gz.xacro (robot description, xacro)
@@ -36,6 +36,6 @@
                 <box size="0.05 0.05 0.05"/>
             </geometry>
-            <material name="blue">
-                <color rgba="0.0 0.0 1.0 1.0"/>
+            <material name="red">
+                <color rgba="1.0 0.0 0.0 1.0"/>
             </material>
         </visual>
@@ -45,4 +45,9 @@
             </geometry>
         </collision>
+        <sensor name='sensor_contact' type='contact'>
+            <contact>
+                <collision>collision</collision>
+            </contact>
+        </sensor>
     </link>
         <!-- <plugin name="gz::sim::systems::OdometryPublisher" filename="gz-sim-odometry-publisher-system">
@@ -53,23 +58,46 @@
             <tf_topic>/tf</tf_topic>
         </plugin> -->
-<!--
+    <gazebo>
         <plugin name="gz::sim::systems::DetachableJoint" filename="gz-sim-detachable-joint-system">
             <parent_link>col_gripper</parent_link>
             <child_model>cylinder11</child_model>
             <child_link>cylinder1_link</child_link>
-        </plugin> -->
-    <gazebo>
-        <plugin filename="gz-sim-touchplugin-system" name="gz::sim::systems::TouchPlugin">
-            <target>48</target>
+            <attach_topic>/model/cylinder11/detachable_joint/attach</attach_topic>
+            <detach_topic>/model/cylinder11/detachable_joint/detach</detach_topic>
+        </plugin>
+        <!-- <plugin filename="gz-sim-touchplugin-system" name="gz::sim::systems::TouchPlugin">
+            <target>cylinder11</target>
+            <link_name>gripper_trigger</link_name>
             <namespace>trigger</namespace>
             <time>0.001</time>
             <enabled>true</enabled>
+        </plugin> -->
+        <!-- <plugin filename="gz-sim-contact-system"
+            name="gz::sim::systems::Contact">
         </plugin>
-        <!-- <plugin filename="gz-sim-triggered-publisher-system" name="gz::sim::systems::TriggeredPublisher">
-            <input type="gz.msgs.Boolean" topic="/trigger/touched">
+        <plugin filename="gz-sim-touchplugin-system"
+        name="gz::sim::systems::TouchPlugin">
+            <target>cylinder</target>
+            <namespace>gripper_trigger</namespace>
+            <time>0.001</time>
+            <enabled>true</enabled>
+        </plugin>
+ -->
+        <plugin filename="gz-sim-triggered-publisher-system" name="gz::sim::systems::TriggeredPublisher">
+            <input type="gz.msgs.Boolean" topic="/attach_topic">
             <match>data: true</match>
             </input>
-            <output type="gz.msgs.Empty" topic="/cylinder1/detach"/>
-        </plugin> -->
+            <output type="gz.msgs.Empty" topic="/model/cylinder11/detachable_joint/attach">
+                unused: true
+            </output>
+        </plugin>
+        <plugin filename="gz-sim-triggered-publisher-system" name="gz::sim::systems::TriggeredPublisher">
+            <input type="gz.msgs.Boolean" topic="/detach_topic">
+            <match>data: true</match>
+            </input>
+            <output type="gz.msgs.Empty" topic="/model/cylinder11/detachable_joint/detach">
+                unused: true
+            </output>
+        </plugin>
         <!-- <plugin filename="gz-sim-detachable-joint-system" name="gz::sim::systems::DetachableJoint">
             <parent_link>col_gripper</parent_link>
@@ -93,4 +121,6 @@
             <cmd_min>-1000</cmd_min>
         </plugin>
+        <!-- <plugin name="gz::sim::systems::DetachableJoint">
+        </plugin> -->
     </gazebo>
 </robot>

Commit message: grip_test and util.Gripper

File: src/shesnar/urdf/sim_gripper_gz.xacro (robot description, xacro)
@@ -45,9 +45,4 @@
             </geometry>
         </collision>
-        <sensor name='sensor_contact' type='contact'>
-            <contact>
-                <collision>collision</collision>
-            </contact>
-        </sensor>
     </link>
         <!-- <plugin name="gz::sim::systems::OdometryPublisher" filename="gz-sim-odometry-publisher-system">
@@ -61,14 +56,28 @@
         <plugin name="gripper_plugin_gz::DynamicDetachableJoint" filename="libgripper_plugin_gz.so">
             <parent_link>col_gripper</parent_link>
-            <attach_topic>/model/my_bot/detachable_joint1/attach</attach_topic>
-            <detach_topic>/model/my_bot/detachable_joint1/detach</detach_topic>
-            <output_topic>/model/my_bot/detachable_joint1/output</output_topic>
+            <attach_topic>/detachable_jointcl/attach</attach_topic>
+            <detach_topic>/detachable_jointcl/detach</detach_topic>
+            <output_topic>/detachable_jointcl/output</output_topic>
             <!-- <grip_link>cylinder1_link</grip_link> -->
         </plugin>
         <plugin name="gripper_plugin_gz::DynamicDetachableJoint" filename="libgripper_plugin_gz.so">
             <parent_link>col_gripper</parent_link>
-            <attach_topic>/model/my_bot/detachable_joint2/attach</attach_topic>
-            <detach_topic>/model/my_bot/detachable_joint2/detach</detach_topic>
-            <output_topic>/model/my_bot/detachable_joint2/output</output_topic>
+            <attach_topic>/detachable_jointcr/attach</attach_topic>
+            <detach_topic>/detachable_jointcr/detach</detach_topic>
+            <output_topic>/detachable_jointcr/output</output_topic>
+            <!-- <grip_link>cylinder1_link</grip_link> -->
+        </plugin>
+        <plugin name="gripper_plugin_gz::DynamicDetachableJoint" filename="libgripper_plugin_gz.so">
+            <parent_link>col_gripper</parent_link>
+            <attach_topic>/detachable_jointsl/attach</attach_topic>
+            <detach_topic>/detachable_jointsl/detach</detach_topic>
+            <output_topic>/detachable_jointsl/output</output_topic>
+            <!-- <grip_link>cylinder1_link</grip_link> -->
+        </plugin>
+        <plugin name="gripper_plugin_gz::DynamicDetachableJoint" filename="libgripper_plugin_gz.so">
+            <parent_link>col_gripper</parent_link>
+            <attach_topic>/detachable_jointsr/attach</attach_topic>
+            <detach_topic>/detachable_jointsr/detach</detach_topic>
+            <output_topic>/detachable_jointsr/output</output_topic>
             <!-- <grip_link>cylinder1_link</grip_link> -->
         </plugin>
@@ -99,20 +108,4 @@
         </plugin>
  -->
-        <plugin filename="gz-sim-triggered-publisher-system" name="gz::sim::systems::TriggeredPublisher">
-            <input type="gz.msgs.Boolean" topic="/attach_topic">
-            <match>data: true</match>
-            </input>
-            <output type="gz.msgs.Empty" topic="/model/cylinder11/detachable_joint/attach">
-                unused: true
-            </output>
-        </plugin>
-        <plugin filename="gz-sim-triggered-publisher-system" name="gz::sim::systems::TriggeredPublisher">
-            <input type="gz.msgs.Boolean" topic="/detach_topic">
-            <match>data: true</match>
-            </input>
-            <output type="gz.msgs.Empty" topic="/model/cylinder11/detachable_joint/detach">
-                unused: true
-            </output>
-        </plugin>
         <!-- <plugin filename="gz-sim-detachable-joint-system" name="gz::sim::systems::DetachableJoint">
             <parent_link>col_gripper</parent_link>

Commit message: grip_test and util.Gripper

File: src/shesnar/urdf/sim_gripper_gz.xacro (robot description, xacro)
@@ -45,9 +45,4 @@
             </geometry>
         </collision>
-        <sensor name='sensor_contact' type='contact'>
-            <contact>
-                <collision>collision</collision>
-            </contact>
-        </sensor>
     </link>
  -->
@@ -84,14 +79,28 @@
         <plugin name="gripper_plugin_gz::DynamicDetachableJoint" filename="libgripper_plugin_gz.so">
             <parent_link>col_gripper</parent_link>
-            <attach_topic>/model/my_bot/detachable_joint1/attach</attach_topic>
-            <detach_topic>/model/my_bot/detachable_joint1/detach</detach_topic>
-            <output_topic>/model/my_bot/detachable_joint1/output</output_topic>
+            <attach_topic>/detachable_jointcl/attach</attach_topic>
+            <detach_topic>/detachable_jointcl/detach</detach_topic>
+            <output_topic>/detachable_jointcl/output</output_topic>
             <!-- <grip_link>cylinder1_link</grip_link> -->
         </plugin>
         <plugin name="gripper_plugin_gz::DynamicDetachableJoint" filename="libgripper_plugin_gz.so">
             <parent_link>col_gripper</parent_link>
-            <attach_topic>/model/my_bot/detachable_joint2/attach</attach_topic>
-            <detach_topic>/model/my_bot/detachable_joint2/detach</detach_topic>
-            <output_topic>/model/my_bot/detachable_joint2/output</output_topic>
+            <attach_topic>/detachable_jointcr/attach</attach_topic>
+            <detach_topic>/detachable_jointcr/detach</detach_topic>
+            <output_topic>/detachable_jointcr/output</output_topic>
+            <!-- <grip_link>cylinder1_link</grip_link> -->
+        </plugin>
+        <plugin name="gripper_plugin_gz::DynamicDetachableJoint" filename="libgripper_plugin_gz.so">
+            <parent_link>col_gripper</parent_link>
+            <attach_topic>/detachable_jointsl/attach</attach_topic>
+            <detach_topic>/detachable_jointsl/detach</detach_topic>
+            <output_topic>/detachable_jointsl/output</output_topic>
+            <!-- <grip_link>cylinder1_link</grip_link> -->
+        </plugin>
+        <plugin name="gripper_plugin_gz::DynamicDetachableJoint" filename="libgripper_plugin_gz.so">
+            <parent_link>col_gripper</parent_link>
+            <attach_topic>/detachable_jointsr/attach</attach_topic>
+            <detach_topic>/detachable_jointsr/detach</detach_topic>
+            <output_topic>/detachable_jointsr/output</output_topic>
             <!-- <grip_link>cylinder1_link</grip_link> -->
         </plugin>
