Commit message: Added lifters_control

File: src/shesnar/urdf/robot_lifters.xacro (robot description, xacro)
@@ -59,5 +59,9 @@
         <origin xyz="0.0 0.0 0.07" rpy="0 0 0"/>
         <axis xyz="0 0 1"/>
+<<<<<<< HEAD
         <limit effort="1000.0" lower="0" upper="0.2" velocity="0.5"/>
+=======
+        <limit effort="1000.0" lower="0" upper="0.11" velocity="0.5"/>
+>>>>>>> b3c9261 (Added lifters_control)
     </joint>
     <!-- Revolute Joint 1 (вращение банки 1) -->
@@ -90,4 +94,15 @@
         <origin xyz="0.05 0 0.05" rpy="0 0 0"/>
     </joint> -->
+<<<<<<< HEAD
+=======
+    <joint name="can_rotator_1_joint" type="revolute">
+        <parent link="can_lift_link"/>
+        <child link="can_rotator_1_link"/>
+        <origin xyz="0 0.05 0" rpy="0 0 0"/>
+        <axis xyz="0 0 1"/>
+        <limit lower="-1.57" upper="1.57" effort="5" velocity="7.0"/>
+        <dynamics damping="0.1"/>
+    </joint>
+>>>>>>> b3c9261 (Added lifters_control)
     <!-- Revolute Joint 2 (вращение банки 2) -->
     <!-- <link name="can_rotator_2_link">
@@ -108,5 +123,9 @@
             <material name="blue">
                 <color rgba="0.0 0.0 1.0 1.0"/>
+<<<<<<< HEAD
             </material>                                                     завхват банки №2
+=======
+            </material>                                                       <!-- завхват банки №2 -->
+>>>>>>> b3c9261 (Added lifters_control)
         </visual>
         <xacro:inertial_box mass="0.1" x="0.05" y="0.05" z='0.05'>
@@ -173,3 +192,65 @@
         </plugin>
     </gazebo>
+    <joint name="can_rotator_2_joint" type="revolute">
+        <parent link="can_lift_link"/>
+        <child link="can_rotator_2_link"/>
+        <origin xyz="0 -0.05 0" rpy="0 0 0"/>
+        <axis xyz="0 0 -1"/>
+        <limit lower="-1.57" upper="1.57" effort="5" velocity="7.0"/>
+         <dynamics damping="0.1"/>
+    </joint>
+      <gazebo>
+        <plugin name="gz::sim::systems::JointStatePublisher" filename="gz-sim-joint-state-publisher-system">
+            <!-- <joint_name>board_lift_joint</joint_name>
+            <joint_name>can_lift_joint</joint_name>
+            <joint_name>can_rotator_1_joint</joint_name>
+            <joint_name>can_rotator_2_joint</joint_name> -->
+        </plugin>
+        <plugin name="gz::sim::systems::JointPositionController" filename="gz-sim-joint-position-controller-system">
+            <topic>board_lift_topic</topic>
+            <joint_name>board_lift_joint</joint_name>
+            <!-- <joint_index>1</joint_index> -->
+            <p_gain>100</p_gain>
+            <i_gain>0.1</i_gain>
+            <d_gain>10.0</d_gain>
+            <i_max>1</i_max>
+            <i_min>-1</i_min>
+            <cmd_max>50000</cmd_max>
+            <cmd_min>-50000</cmd_min>
+        </plugin>
+        <plugin name="gz::sim::systems::JointPositionController" filename="gz-sim-joint-position-controller-system">
+            <topic>can_lift_topic</topic>
+            <joint_name>can_lift_joint</joint_name>
+            <!-- <joint_index>1</joint_index> -->
+            <p_gain>100</p_gain>
+            <i_gain>0.1</i_gain>
+            <d_gain>10.0</d_gain>
+            <i_max>1</i_max>
+            <i_min>-1</i_min>
+            <cmd_max>50000</cmd_max>
+            <cmd_min>-50000</cmd_min>
+        </plugin>
+        <plugin name="gz::sim::systems::JointPositionController" filename="gz-sim-joint-position-controller-system">
+            <topic>can_rotator_1_topic</topic>
+            <joint_name>can_rotator_1_joint</joint_name>
+            <p_gain>10</p_gain>
+            <i_gain>0.1</i_gain>
+            <d_gain>0.01</d_gain>
+            <i_max>1</i_max>
+            <i_min>-1</i_min>
+            <cmd_max>1000</cmd_max>
+            <cmd_min>-1000</cmd_min>
+        </plugin>
+        <plugin name="gz::sim::systems::JointPositionController" filename="gz-sim-joint-position-controller-system">
+            <topic>can_rotator_2_topic</topic>
+            <joint_name>can_rotator_2_joint</joint_name>
+            <p_gain>10</p_gain>
+            <i_gain>0.1</i_gain>
+            <d_gain>0.01</d_gain>
+            <i_max>1</i_max>
+            <i_min>-1</i_min>
+            <cmd_max>1000</cmd_max>
+            <cmd_min>-1000</cmd_min>
+        </plugin>
+    </gazebo>
 </robot>

Commit message: Added lifters_control

File: src/shesnar/urdf/robot_lifters.xacro (robot description, xacro)
@@ -7,5 +7,7 @@
                 <box size="0.025 0.025 0.025"/>
             </geometry>
-            <material name="red"/>
+            <material name="red">
+                <color rgba="1.0 0.0 0.0 1.0"/>
+            </material>
         </visual>
         <xacro:inertial_box mass="0.2" x="0.025" y="0.025" z='0.025'>
@@ -18,5 +20,7 @@
                 <box size="0.03 0.03 0.03"/>
             </geometry>
-            <material name="blue"/>             <!--захват доски прикрепленный к prismatic 1 и отвечающий за подъем доски-->
+            <material name="blue">                     <!--захват доски прикрепленный к prismatic 1 и отвечающий за подъем доски-->
+                <color rgba="0.0 0.0 1.0 1.0"/>
+            </material>
         </visual>
         <xacro:inertial_box mass="0.1" x="0.05" y="0.05" z='0.05'>
@@ -34,5 +38,5 @@
         <origin xyz="0 0 0.14" rpy="0 0 0"/>
         <axis xyz="0 0 1"/>
-        <limit lower="0" upper="0.11" effort="10" velocity="0.1"/>
+        <limit lower="0" upper="0.11" effort="1000.0" velocity="0.5"/>
     </joint>
     <!-- Prismatic Joint 2 (подъём банок) -->
@@ -42,5 +46,7 @@
                <box size="0.025 0.025 0.025"/>
             </geometry>
-            <material name="blue"/>
+            <material name="blue">
+                <color rgba="0.0 0.0 1.0 1.0"/>
+            </material>
         </visual>
         <xacro:inertial_box mass="0.2" x="0.025" y="0.025" z='0.025'>
@@ -53,5 +59,5 @@
         <origin xyz="0.1 0.0 0.028" rpy="0 0 0"/>
         <axis xyz="0 0 1"/>
-        <limit lower="0" upper="0.11" effort="10" velocity="0.1"/>
+        <limit effort="1000.0" lower="0" upper="0.11" velocity="0.5"/>
     </joint>
     <!-- Revolute Joint 1 (вращение банки 1) -->
@@ -61,5 +67,7 @@
                 <cylinder radius="0.015" length="0.02"/>
             </geometry>
-            <material name="red"/>
+            <material name="red">
+                <color rgba="1.0 0.0 0.0 1.0"/>
+            </material>
         </visual>
     </link>
@@ -69,5 +77,7 @@
                 <box size="0.03 0.03 0.03"/>                      <!-- завхват банки №1 -->
             </geometry>
-            <material name="blue"/>
+            <material name="blue">
+                <color rgba="0.0 0.0 1.0 1.0"/>
+            </material>
         </visual>
         <xacro:inertial_box mass="0.1" x="0.05" y="0.05" z='0.05'>
@@ -85,5 +95,5 @@
         <origin xyz="0 0.05 0" rpy="0 0 0"/>
         <axis xyz="0 0 1"/>
-        <limit lower="-1.57" upper="1.57" effort="5" velocity="0.5"/>
+        <limit lower="-1.57" upper="1.57" effort="5" velocity="7.0"/>
         <dynamics damping="0.1"/>
     </joint>
@@ -94,5 +104,7 @@
                 <cylinder radius="0.015" length="0.02"/>
             </geometry>
-            <material name="red"/>
+            <material name="red">
+                <color rgba="1.0 0.0 0.0 1.0"/>
+            </material>
         </visual>
     </link>
@@ -102,5 +114,7 @@
                 <box size="0.03 0.03 0.03"/>
             </geometry>
-            <material name="blue"/>                                                       <!-- завхват банки №2 -->
+            <material name="blue">
+                <color rgba="0.0 0.0 1.0 1.0"/>
+            </material>                                                       <!-- завхват банки №2 -->
         </visual>
         <xacro:inertial_box mass="0.1" x="0.05" y="0.05" z='0.05'>
@@ -117,7 +131,61 @@
         <child link="can_rotator_2_link"/>
         <origin xyz="0 -0.05 0" rpy="0 0 0"/>
-        <axis xyz="0 0 1"/>
-        <limit lower="-1.57" upper="1.57" effort="5" velocity="0.5"/>
+        <axis xyz="0 0 -1"/>
+        <limit lower="-1.57" upper="1.57" effort="5" velocity="7.0"/>
          <dynamics damping="0.1"/>
     </joint>
+      <gazebo>
+        <plugin name="gz::sim::systems::JointStatePublisher" filename="gz-sim-joint-state-publisher-system">
+            <!-- <joint_name>board_lift_joint</joint_name>
+            <joint_name>can_lift_joint</joint_name>
+            <joint_name>can_rotator_1_joint</joint_name>
+            <joint_name>can_rotator_2_joint</joint_name> -->
+        </plugin>
+        <plugin name="gz::sim::systems::JointPositionController" filename="gz-sim-joint-position-controller-system">
+            <topic>board_lift_topic</topic>
+            <joint_name>board_lift_joint</joint_name>
+            <!-- <joint_index>1</joint_index> -->
+            <p_gain>100</p_gain>
+            <i_gain>0.1</i_gain>
+            <d_gain>10.0</d_gain>
+            <i_max>1</i_max>
+            <i_min>-1</i_min>
+            <cmd_max>50000</cmd_max>
+            <cmd_min>-50000</cmd_min>
+        </plugin>
+        <plugin name="gz::sim::systems::JointPositionController" filename="gz-sim-joint-position-controller-system">
+            <topic>can_lift_topic</topic>
+            <joint_name>can_lift_joint</joint_name>
+            <!-- <joint_index>1</joint_index> -->
+            <p_gain>100</p_gain>
+            <i_gain>0.1</i_gain>
+            <d_gain>10.0</d_gain>
+            <i_max>1</i_max>
+            <i_min>-1</i_min>
+            <cmd_max>50000</cmd_max>
+            <cmd_min>-50000</cmd_min>
+        </plugin>
+        <plugin name="gz::sim::systems::JointPositionController" filename="gz-sim-joint-position-controller-system">
+            <topic>can_rotator_1_topic</topic>
+            <joint_name>can_rotator_1_joint</joint_name>
+            <p_gain>10</p_gain>
+            <i_gain>0.1</i_gain>
+            <d_gain>0.01</d_gain>
+            <i_max>1</i_max>
+            <i_min>-1</i_min>
+            <cmd_max>1000</cmd_max>
+            <cmd_min>-1000</cmd_min>
+        </plugin>
+        <plugin name="gz::sim::systems::JointPositionController" filename="gz-sim-joint-position-controller-system">
+            <topic>can_rotator_2_topic</topic>
+            <joint_name>can_rotator_2_joint</joint_name>
+            <p_gain>10</p_gain>
+            <i_gain>0.1</i_gain>
+            <d_gain>0.01</d_gain>
+            <i_max>1</i_max>
+            <i_min>-1</i_min>
+            <cmd_max>1000</cmd_max>
+            <cmd_min>-1000</cmd_min>
+        </plugin>
+    </gazebo>
 </robot>
