Commit message: xacro uptate

File: src/shesnar/urdf/robot_core.xacro (robot description, xacro)
@@ -25,6 +25,6 @@
             <origin xyz="-0.18 -0.1 0" rpy="0 0 0" />
             <geometry>
-                <mesh filename="package://shesnar/meshes/body.dae" scale="0.001 0.001 0.001" rpy="0 0 1.04"/>
-            <!-- <cylinder radius="0.20" length="0.12"/> -->
+            <!-- <mesh filename="package://shesnar/meshes/body.dae" scale="0.001 0.001 0.001" rpy="0 0 1.04"/> -->
+                <mesh filename="file://$(find shesnar)/meshes/body.dae" scale="0.001 0.001 0.001" rpy="0 0 1.04"/>
             </geometry>
             <material name="">

Commit message: little update

File: src/shesnar/urdf/robot_core.xacro (robot description, xacro)
@@ -23,5 +23,5 @@
     <link name="body">
         <visual>
-            <origin xyz="-0.18 -0.1 0" rpy="0 0 0" />
+            <origin xyz="0.1 -0.18 0" rpy="0 0 1.57" />
             <geometry>
                 <mesh filename="package://shesnar/meshes/body.dae" scale="0.001 0.001 0.001" rpy="0 0 1.04"/>

Commit message: little fixes

File: src/shesnar/urdf/robot_core.xacro (robot description, xacro)
@@ -23,7 +23,7 @@
     <link name="body">
         <visual>
-            <origin xyz="0.1 -0.18 0" rpy="0 0 1.57" />
+            <origin xyz="0.1 -0.18 0" rpy="1.57 0 1.57" />
             <geometry>
-                <mesh scale="0.001 0.001 0.001" rpy="0 0 1.04" filename="file://$(find shesnar)/meshes/body.obj"/>
+                <mesh scale="0.1 0.1 0.1" rpy="0 0 1.04" filename="file://$(find shesnar)/meshes/body.obj"/>
             <!-- <cylinder radius="0.20" length="0.12"/> -->
             </geometry>
@@ -33,7 +33,8 @@
         </visual>
         <collision>
-            <origin xyz="0 0 0.06" rpy="0 0 0" />
+            <origin xyz="0.1 -0.18 0" rpy="1.57 0 1.57" />
             <geometry>
-                <cylinder radius="0.20" length="0.12"/>
+                 <mesh scale="0.1 0.1 0.1" rpy="0 0 1.04" filename="file://$(find shesnar)/meshes/body_collision.obj"/>
+                <!-- <cylinder radius="0.20" length="0.12"/> -->
             </geometry>
         </collision>

Commit message: add odom

File: src/shesnar/urdf/robot_core.xacro (robot description, xacro)
@@ -9,7 +9,14 @@
     </material>
     <xacro:include filename="inertial_macros.xacro"/>
+    <link name="odom"></link>
+    <joint name="odom_joint" type="fixed">
+        <parent link="odom"/>
+        <child link="base_link"/>
+        <origin xyz="0 0 0"/>
+    </joint>
     <link name="base_link"></link>
     <joint name="body_joint" type="fixed">
-        <parent link="base_link"/>
+        <!-- <parent link="base_link"/> -->
+        <parent link="odom"/>
         <child link="body"/>
         <origin xyz="0 0 0"/>
@@ -44,5 +51,5 @@
     </link>
       <gazebo>
-        <!-- <plugin name="gz::sim::systems::OdometryPublisher" filename="gz-sim-odometry-publisher-system">
+        <plugin name="gz::sim::systems::OdometryPublisher" filename="gz-sim-odometry-publisher-system">
             <odom_frame>odom</odom_frame>
             <robot_base_frame>base_link</robot_base_frame>
@@ -50,5 +57,5 @@
             <odom_topic>/odom</odom_topic>
             <tf_topic>/tf</tf_topic>
-        </plugin> -->
+        </plugin>
         <plugin name="gz::sim::systems::VelocityControl" filename="gz-sim-velocity-control-system">
         </plugin>

Commit message: finally fixed tf tree with odom

File: src/shesnar/urdf/robot_core.xacro (robot description, xacro)
@@ -9,14 +9,8 @@
     </material>
     <xacro:include filename="inertial_macros.xacro"/>
-    <link name="odom"></link>
-    <joint name="odom_joint" type="fixed">
-        <parent link="odom"/>
-        <child link="base_link"/>
-        <origin xyz="0 0 0"/>
-    </joint>
+    <!-- <link name="odom"></link> -->
     <link name="base_link"></link>
     <joint name="body_joint" type="fixed">
-        <!-- <parent link="base_link"/> -->
-        <parent link="odom"/>
+        <parent link="base_link"/>
         <child link="body"/>
         <origin xyz="0 0 0"/>
@@ -51,5 +45,5 @@
     </link>
       <gazebo>
-        <plugin name="gz::sim::systems::OdometryPublisher" filename="gz-sim-odometry-publisher-system">
+        <!-- <plugin name="gz::sim::systems::OdometryPublisher" filename="gz-sim-odometry-publisher-system">
             <odom_frame>odom</odom_frame>
             <robot_base_frame>base_link</robot_base_frame>
@@ -57,5 +51,5 @@
             <odom_topic>/odom</odom_topic>
             <tf_topic>/tf</tf_topic>
-        </plugin>
+        </plugin> -->
         <plugin name="gz::sim::systems::VelocityControl" filename="gz-sim-velocity-control-system">
         </plugin>

Commit message: some changes

File: src/shesnar/urdf/robot_core.xacro (robot description, xacro)
@@ -5,9 +5,19 @@
     <compiler meshdir="meshes" discardvisual="false" />
   </mujoco> -->
+      <gazebo>
+        <!-- <plugin name="gz::sim::systems::OdometryPublisher" filename="gz-sim-odometry-publisher-system">
+            <odom_frame>odom</odom_frame>
+            <robot_base_frame>base_link</robot_base_frame>
+            <odom_publish_frequency>50</odom_publish_frequency>
+            <odom_topic>/odom</odom_topic>
+            <tf_topic>/tf</tf_topic>
+        </plugin> -->
+        <plugin name="gz::sim::systems::VelocityControl" filename="gz-sim-velocity-control-system">
+        </plugin>
+    </gazebo>
     <material name="white">
         <color rgba="1 1 1 1" />
     </material>
     <xacro:include filename="inertial_macros.xacro"/>
-    <!-- <link name="odom"></link> -->
     <link name="base_link"></link>
     <joint name="body_joint" type="fixed">
@@ -44,14 +54,3 @@
         </xacro:inertial_cylinder>
     </link>
-      <gazebo>
-        <!-- <plugin name="gz::sim::systems::OdometryPublisher" filename="gz-sim-odometry-publisher-system">
-            <odom_frame>odom</odom_frame>
-            <robot_base_frame>base_link</robot_base_frame>
-            <odom_publish_frequency>50</odom_publish_frequency>
-            <odom_topic>/odom</odom_topic>
-            <tf_topic>/tf</tf_topic>
-        </plugin> -->
-        <plugin name="gz::sim::systems::VelocityControl" filename="gz-sim-velocity-control-system">
-        </plugin>
-    </gazebo>
 </robot>

Commit message: new body

File: src/shesnar/urdf/robot_core.xacro (robot description, xacro)
@@ -36,5 +36,5 @@
             <origin xyz="0.1 -0.18 0" rpy="1.57 0 1.57" />
             <geometry>
-                <mesh scale="0.1 0.1 0.1" rpy="0 0 1.04" filename="file://$(find shesnar)/meshes/body.obj"/>
+                <mesh scale="0.1 0.1 0.1" rpy="0 0 1.04" filename="file://$(find shesnar)/meshes/body2.obj"/>
             <!-- <cylinder radius="0.20" length="0.12"/> -->
             </geometry>
@@ -46,5 +46,5 @@
             <origin xyz="0.1 -0.18 0" rpy="1.57 0 1.57" />
             <geometry>
-                 <mesh scale="0.1 0.1 0.1" rpy="0 0 1.04" filename="file://$(find shesnar)/meshes/body_collision.obj"/>
+                 <mesh scale="0.1 0.1 0.1" rpy="0 0 1.04" filename="file://$(find shesnar)/meshes/body2.obj"/>
                 <!-- <cylinder radius="0.20" length="0.12"/> -->
             </geometry>
