Commit message: Actual version

File: src/shesnar/urdf/robot.urdf.xacro (robot description, xacro)
@@ -5,3 +5,4 @@
     <!-- <xacro:include filename="gripper.xacro"/>  -->
     <xacro:include filename="sim_gripper_gz.xacro"/>
+    <!-- <xacro:include filename="depth_camera.xacro"/>  -->
 </robot>

File: src/shesnar/urdf/sim_gripper_gz.xacro (robot description, xacro)
@@ -42,12 +42,7 @@
         <collision>
             <geometry>
-                <box size="0.05 0.05 0.05"/>
+                <box size="0.06 0.06 0.06"/>
             </geometry>
         </collision>
-      <sensor name='sensor_contact' type='contact'>
-        <contact>
-          <collision>c1</collision>
-        </contact>
-      </sensor>
     </link>
         <!-- <plugin name="gz::sim::systems::OdometryPublisher" filename="gz-sim-odometry-publisher-system">
@@ -66,21 +61,21 @@
     <gazebo>
         <plugin filename="gz-sim-touchplugin-system" name="gz::sim::systems::TouchPlugin">
-            <target>cylinder11</target>
+            <target>48</target>
             <namespace>trigger</namespace>
             <time>0.001</time>
             <enabled>true</enabled>
         </plugin>
-        <plugin filename="gz-sim-triggered-publisher-system" name="gz::sim::systems::TriggeredPublisher">
+        <!-- <plugin filename="gz-sim-triggered-publisher-system" name="gz::sim::systems::TriggeredPublisher">
             <input type="gz.msgs.Boolean" topic="/trigger/touched">
             <match>data: true</match>
             </input>
             <output type="gz.msgs.Empty" topic="/cylinder1/detach"/>
-        </plugin>
-        <plugin filename="gz-sim-detachable-joint-system" name="gz::sim::systems::DetachableJoint">
+        </plugin> -->
+        <!-- <plugin filename="gz-sim-detachable-joint-system" name="gz::sim::systems::DetachableJoint">
             <parent_link>col_gripper</parent_link>
             <child_model>cylinder11</child_model>
             <child_link>cylinder1_link</child_link>
             <detach_topic>/cylinder1/detach</detach_topic>
-        </plugin>
+        </plugin> -->
         <plugin name="gz::sim::systems::JointStatePublisher" filename="gz-sim-joint-state-publisher-system">
             <!-- <topic>joint_states</topic>  -->

Commit message: some trubles

File: src/shesnar/urdf/robot.urdf.xacro (robot description, xacro)
@@ -2,8 +2,7 @@
 <robot xmlns:xacro="http://www.ros.org/wiki/xacro"  name="neuro_korch">
     <xacro:include filename="robot_core.xacro"/>
-    <xacro:include filename="lidar.xacro"/>
+    <!-- <xacro:include filename="lidar.xacro"/>
     <xacro:include filename="robot_lifters.xacro"/>
-    <!-- <xacro:include filename="sim_gripper_gz.xacro"/>  -->
-    <xacro:include filename="can_gripper.xacro"/>
+    <xacro:include filename="can_gripper.xacro"/>  -->
     <!-- <xacro:include filename="depth_camera.xacro"/>  -->
 </robot>

File: src/shesnar/urdf/robot_core.xacro (robot description, xacro)
@@ -16,4 +16,79 @@
         </plugin>
     </gazebo>
+    <!-- <link name="caster_1">
+        <collision>
+            <geometry>
+                <sphere radius="0.005" />
+            </geometry>
+            <surface>
+                <friction>
+                    <ode>
+                    <mu>0.00001</mu>
+                    <mu2>0.00001</mu2>
+                    </ode>
+                </friction>
+             </surface>
+        </collision>
+        <visual>
+            <geometry>
+            <sphere radius="0.005" />
+            </geometry>
+        </visual>
+    </link>
+    <joint name="caster_1_joint" type="fixed">
+        <parent link="base_link"/>
+        <child link="caster_1"/>
+        <origin xyz="0.08 0.12 -0.01"/>
+    </joint>
+    <link name="caster_2">
+        <collision>
+            <geometry>
+                <sphere radius="0.005" />
+            </geometry>
+            <surface>
+                <friction>
+                    <ode>
+                    <mu>0.00001</mu>
+                    <mu2>0.00001</mu2>
+                    </ode>
+                </friction>
+             </surface>
+        </collision>
+        <visual>
+            <geometry>
+            <sphere radius="0.005" />
+            </geometry>
+        </visual>
+    </link>
+    <joint name="caster_2_joint" type="fixed">
+        <parent link="base_link"/>
+        <child link="caster_2"/>
+        <origin xyz="0.08 -0.12 -0.01"/>
+    </joint>
+   <link name="caster_3">
+        <collision>
+            <geometry>
+                <sphere radius="0.005" />
+            </geometry>
+            <surface>
+                <friction>
+                    <ode>
+                    <mu>0.00001</mu>
+                    <mu2>0.00001</mu2>
+                    </ode>
+                </friction>
+             </surface>
+        </collision>
+        <visual>
+            <geometry>
+            <sphere radius="0.005" />
+            </geometry>
+        </visual>
+    </link>
+    <joint name="caster_3_joint" type="fixed">
+        <parent link="base_link"/>
+        <child link="caster_3"/>
+        <origin xyz="-0.1 0.0 -0.01"/>
+    </joint> -->
     <material name="white">
         <color rgba="1 1 1 1" />
@@ -34,7 +109,7 @@
     <link name="body">
         <visual>
-            <origin xyz="0.1 -0.18 0" rpy="1.57 0 1.57" />
+            <origin xyz="0.1 -0.1759 0" rpy="1.57 0 1.57" />
             <geometry>
-                <mesh scale="0.1 0.1 0.1" rpy="0 0 1.04" filename="file://$(find shesnar)/meshes/body2.obj"/>
+                <mesh scale="0.1 0.1 0.1" rpy="0 0 1.04" filename="file://$(find shesnar)/meshes/body.obj"/>
             <!-- <cylinder radius="0.20" length="0.12"/> -->
             </geometry>
@@ -44,11 +119,11 @@
         </visual>
         <collision>
-            <origin xyz="0.1 -0.18 0" rpy="1.57 0 1.57" />
+            <origin xyz="0.1 -0.1759 0" rpy="1.57 0 1.57" />
             <geometry>
-                 <mesh scale="0.1 0.1 0.1" rpy="0 0 1.04" filename="file://$(find shesnar)/meshes/body2.obj"/>
+                 <mesh scale="0.1 0.1 0.1" rpy="0 0 1.04" filename="file://$(find shesnar)/meshes/body.obj"/>
                 <!-- <cylinder radius="0.20" length="0.12"/> -->
             </geometry>
         </collision>
-        <xacro:inertial_cylinder mass="4.0" length="0.12" radius="0.15">
+        <xacro:inertial_cylinder mass="10.0" length="0.12" radius="0.15">
             <origin xyz="0 0 0" rpy="0 0 0"/>
         </xacro:inertial_cylinder>

Commit message: fix rotating issue

File: src/shesnar/urdf/robot.urdf.xacro (robot description, xacro)
@@ -2,7 +2,7 @@
 <robot xmlns:xacro="http://www.ros.org/wiki/xacro"  name="neuro_korch">
     <xacro:include filename="robot_core.xacro"/>
-    <!-- <xacro:include filename="lidar.xacro"/>
+    <xacro:include filename="lidar.xacro"/>
     <xacro:include filename="robot_lifters.xacro"/>
-    <xacro:include filename="can_gripper.xacro"/>  -->
+    <xacro:include filename="can_gripper.xacro"/>
     <!-- <xacro:include filename="depth_camera.xacro"/>  -->
 </robot>

File: src/shesnar/urdf/robot_core.xacro (robot description, xacro)
@@ -16,5 +16,5 @@
         </plugin>
     </gazebo>
-    <!-- <link name="caster_1">
+    <link name="caster_1">
         <collision>
             <geometry>
@@ -90,5 +90,5 @@
         <child link="caster_3"/>
         <origin xyz="-0.1 0.0 -0.01"/>
-    </joint> -->
+    </joint>
     <material name="white">
         <color rgba="1 1 1 1" />
@@ -111,5 +111,5 @@
             <origin xyz="0.1 -0.1759 0" rpy="1.57 0 1.57" />
             <geometry>
-                <mesh scale="0.1 0.1 0.1" rpy="0 0 1.04" filename="file://$(find shesnar)/meshes/body.obj"/>
+                <mesh scale="0.1 0.1 0.1" rpy="0 0 1.04" filename="file://$(find shesnar)/meshes/body2.obj"/>
             <!-- <cylinder radius="0.20" length="0.12"/> -->
             </geometry>
@@ -121,5 +121,5 @@
             <origin xyz="0.1 -0.1759 0" rpy="1.57 0 1.57" />
             <geometry>
-                 <mesh scale="0.1 0.1 0.1" rpy="0 0 1.04" filename="file://$(find shesnar)/meshes/body.obj"/>
+                 <mesh scale="0.1 0.1 0.1" rpy="0 0 1.04" filename="file://$(find shesnar)/meshes/body2.obj"/>
                 <!-- <cylinder radius="0.20" length="0.12"/> -->
             </geometry>
