Commit message: merge grip and art urdf

File: src/shesnar/urdf/can_gripper.xacro (robot description, xacro)
@@ -145,4 +145,11 @@
             <grip_link>grip_link</grip_link>
         </plugin>
+        <plugin name="gripper_plugin_gz::DynamicDetachableJoint" filename="libgripper_plugin_gz.so">
+            <parent_link>col_gripper</parent_link>
+            <attach_topic>/detachable_jointsr/attach</attach_topic>
+            <detach_topic>/detachable_jointsr/detach</detach_topic>
+            <output_topic>/detachable_jointsr/output</output_topic>
+            <grip_link>cylinder1_link</grip_link>
+        </plugin> -->
     </gazebo>
 </robot>

File: src/shesnar/urdf/robot_lifters.xacro (robot description, xacro)
@@ -59,9 +59,5 @@
         <origin xyz="0.0 0.0 0.07" rpy="0 0 0"/>
         <axis xyz="0 0 1"/>
-<<<<<<< HEAD
         <limit effort="1000.0" lower="0" upper="0.2" velocity="0.5"/>
-=======
-        <limit effort="1000.0" lower="0" upper="0.11" velocity="0.5"/>
->>>>>>> b3c9261 (Added lifters_control)
     </joint>
     <!-- Revolute Joint 1 (вращение банки 1) -->
@@ -94,4 +90,5 @@
         <origin xyz="0.05 0 0.05" rpy="0 0 0"/>
     </joint> -->
+<<<<<<< HEAD
 <<<<<<< HEAD
 =======
@@ -105,4 +102,6 @@
     </joint>
 >>>>>>> b3c9261 (Added lifters_control)
+=======
+>>>>>>> f41de3b (merge grip and art urdf)
     <!-- Revolute Joint 2 (вращение банки 2) -->
     <!-- <link name="can_rotator_2_link">
@@ -124,8 +123,12 @@
                 <color rgba="0.0 0.0 1.0 1.0"/>
 <<<<<<< HEAD
+<<<<<<< HEAD
             </material>                                                     завхват банки №2
 =======
             </material>                                                       <!-- завхват банки №2 -->
 >>>>>>> b3c9261 (Added lifters_control)
+=======
+            </material>                                                     завхват банки №2
+>>>>>>> f41de3b (merge grip and art urdf)
         </visual>
         <xacro:inertial_box mass="0.1" x="0.05" y="0.05" z='0.05'>
@@ -138,4 +141,5 @@
         <origin xyz="0.05 0 0.05" rpy="0 0 0"/>
     </joint> -->
+<<<<<<< HEAD
       <gazebo>
         <plugin name="gz::sim::systems::JointStatePublisher" filename="gz-sim-joint-state-publisher-system">
@@ -192,12 +196,6 @@
         </plugin>
     </gazebo>
-    <joint name="can_rotator_2_joint" type="revolute">
-        <parent link="can_lift_link"/>
-        <child link="can_rotator_2_link"/>
-        <origin xyz="0 -0.05 0" rpy="0 0 0"/>
-        <axis xyz="0 0 -1"/>
-        <limit lower="-1.57" upper="1.57" effort="5" velocity="7.0"/>
-         <dynamics damping="0.1"/>
-    </joint>
+=======
+>>>>>>> f41de3b (merge grip and art urdf)
       <gazebo>
         <plugin name="gz::sim::systems::JointStatePublisher" filename="gz-sim-joint-state-publisher-system">
@@ -234,5 +232,5 @@
             <topic>can_rotator_1_topic</topic>
             <joint_name>can_rotator_1_joint</joint_name>
-            <p_gain>10</p_gain>
+            <p_gain>100</p_gain>
             <i_gain>0.1</i_gain>
             <d_gain>0.01</d_gain>
@@ -245,5 +243,5 @@
             <topic>can_rotator_2_topic</topic>
             <joint_name>can_rotator_2_joint</joint_name>
-            <p_gain>10</p_gain>
+            <p_gain>100</p_gain>
             <i_gain>0.1</i_gain>
             <d_gain>0.01</d_gain>

File: src/shesnar/urdf/sim_gripper_gz.xacro (robot description, xacro)
@@ -78,23 +78,23 @@
         </plugin>
         <plugin name="gripper_plugin_gz::DynamicDetachableJoint" filename="libgripper_plugin_gz.so">
-            <parent_link>col_gripper</parent_link>
+            <parent_link>can_gripper_1</parent_link>
             <attach_topic>/detachable_jointcl/attach</attach_topic>
             <detach_topic>/detachable_jointcl/detach</detach_topic>
             <output_topic>/detachable_jointcl/output</output_topic>
-            <!-- <grip_link>cylinder1_link</grip_link> -->
+            <grip_link>grip_link</grip_link>
         </plugin>
         <plugin name="gripper_plugin_gz::DynamicDetachableJoint" filename="libgripper_plugin_gz.so">
-            <parent_link>col_gripper</parent_link>
+            <parent_link>can_gripper_2</parent_link>
             <attach_topic>/detachable_jointcr/attach</attach_topic>
             <detach_topic>/detachable_jointcr/detach</detach_topic>
             <output_topic>/detachable_jointcr/output</output_topic>
-            <!-- <grip_link>cylinder1_link</grip_link> -->
+            <grip_link>grip_link</grip_link>
         </plugin>
-        <plugin name="gripper_plugin_gz::DynamicDetachableJoint" filename="libgripper_plugin_gz.so">
+        <!-- <plugin name="gripper_plugin_gz::DynamicDetachableJoint" filename="libgripper_plugin_gz.so">
             <parent_link>col_gripper</parent_link>
             <attach_topic>/detachable_jointsl/attach</attach_topic>
             <detach_topic>/detachable_jointsl/detach</detach_topic>
             <output_topic>/detachable_jointsl/output</output_topic>
-            <!-- <grip_link>cylinder1_link</grip_link> -->
+            <grip_link>cylinder1_link</grip_link>
         </plugin>
         <plugin name="gripper_plugin_gz::DynamicDetachableJoint" filename="libgripper_plugin_gz.so">
@@ -103,5 +103,5 @@
             <detach_topic>/detachable_jointsr/detach</detach_topic>
             <output_topic>/detachable_jointsr/output</output_topic>
-            <!-- <grip_link>cylinder1_link</grip_link> -->
+            <grip_link>cylinder1_link</grip_link>
         </plugin>
 =======

Commit message: merge grip and art urdf

File: src/shesnar/urdf/can_gripper.xacro (robot description, xacro)
@@ -3,5 +3,5 @@
     <link name="can_gripper_1">
         <visual>
-            <origin xyz="0.025 0 0" rpy="0 0 0" />
+            <origin xyz="0.0 0 0.0" rpy="0 0 1.57" />
             <geometry>
                 <box size="0.05 0.02 0.02"/>
@@ -12,5 +12,5 @@
         </visual>
         <collision>
-            <origin xyz="0.025 0 0" rpy="0 0 0" />
+            <origin xyz="0.00 0 0.00" rpy="0 0 1.57" />
             <geometry>
                 <box size="0.05 0.02 0.02"/>
@@ -18,17 +18,17 @@
         </collision>
         <xacro:inertial_box mass="0.01" x="0.05" y="0.02" z="0.02">
-            <origin xyz="0.025 0 0" rpy="0 0 0"/>
+            <origin xyz="0.0 0 0" rpy="0 0 0"/>
         </xacro:inertial_box>
     </link>
-    <joint name="can_gripper_joint_1" type="revolute">
-        <parent link="body"/>
+    <joint name="can_gripper_joint_1" type="prismatic">
+        <parent link="can_lift_link"/>
         <child link="can_gripper_1"/>
-        <origin xyz="0.15 -0.1 0.03" rpy = "0 0 1.57"/>
-        <axis xyz="0 0 -1"/>
-        <limit lower="0.0" upper="3.14" effort="10.0" velocity="7.0"/>
+        <origin xyz="0.05 -0.05 0.05" rpy="0 0 0"/>
+        <axis xyz="1 0 0"/>
+        <limit effort="1000.0" lower="0" upper="0.1" velocity="0.5"/>
     </joint>
     <link name="can_gripper_2">
         <visual>
-            <origin xyz="0.025 0 0" rpy="0 0 0" />
+            <origin xyz="0.0 0 0" rpy="0 0 -1.57" />
             <geometry>
                 <box size="0.05 0.02 0.02"/>
@@ -39,5 +39,5 @@
         </visual>
         <collision>
-            <origin xyz="0.025 0 0" rpy="0 0 0" />
+            <origin xyz="0.0 0 0.0" rpy="0 0 -1.57" />
             <geometry>
                 <box size="0.05 0.02 0.02"/>
@@ -45,45 +45,43 @@
         </collision>
         <xacro:inertial_box mass="0.01" x="0.05" y="0.02" z="0.02">
-            <origin xyz="0.025 0 0" rpy="0 0 0"/>
+            <origin xyz="0.0 0 0" rpy="0 0 0"/>
         </xacro:inertial_box>
     </link>
-    <joint name="can_gripper_joint_2" type="revolute">
-        <parent link="body"/>
+    <joint name="can_gripper_joint_2" type="prismatic">
+        <parent link="can_lift_link"/>
         <child link="can_gripper_2"/>
-        <origin xyz="0.15 0.1 0.03" rpy = "0 0 -1.57"/>
-        <axis xyz="0 0 1"/>
-        <limit lower="0.0" upper="3.14" effort="10.0" velocity="7.0"/>
+        <origin xyz="0.05 0.05 0.05" rpy="0 0 0"/>
+        <axis xyz="1 0 0"/>
+        <limit effort="1000.0" lower="0" upper="0.1" velocity="0.5"/>
     </joint>
     <gazebo>
-        <plugin name="gz::sim::systems::JointStatePublisher" filename="gz-sim-joint-state-publisher-system">
-            <!-- <topic>joint_states</topic>  -->
-            <joint_name>can_gripper_joint_1</joint_name>
+        <plugin name="gripper_plugin_gz::DynamicDetachableJoint" filename="libgripper_plugin_gz.so">
+            <parent_link>can_gripper_1</parent_link>
+            <attach_topic>/detachable_jointcl/attach</attach_topic>
+            <detach_topic>/detachable_jointcl/detach</detach_topic>
+            <output_topic>/detachable_jointcl/output</output_topic>
+            <grip_link>grip_link</grip_link>
         </plugin>
-        <plugin name="gz::sim::systems::JointStatePublisher" filename="gz-sim-joint-state-publisher-system">
-            <!-- <topic>joint_states</topic>  -->
-            <joint_name>can_gripper_joint_2</joint_name>
+        <plugin name="gripper_plugin_gz::DynamicDetachableJoint" filename="libgripper_plugin_gz.so">
+            <parent_link>can_gripper_2</parent_link>
+            <attach_topic>/detachable_jointcr/attach</attach_topic>
+            <detach_topic>/detachable_jointcr/detach</detach_topic>
+            <output_topic>/detachable_jointcr/output</output_topic>
+            <grip_link>grip_link</grip_link>
         </plugin>
-        <plugin name="gz::sim::systems::JointPositionController" filename="gz-sim-joint-position-controller-system">
-            <topic>can_gripper_joint_topic_1</topic>
-            <joint_name>can_gripper_joint_1</joint_name>
-            <p_gain>10</p_gain>
-            <i_gain>0.1</i_gain>
-            <d_gain>0.01</d_gain>
-            <i_max>1</i_max>
-            <i_min>-1</i_min>
-            <cmd_max>1000</cmd_max>
-            <cmd_min>-1000</cmd_min>
+        <!-- <plugin name="gripper_plugin_gz::DynamicDetachableJoint" filename="libgripper_plugin_gz.so">
+            <parent_link>col_gripper</parent_link>
+            <attach_topic>/detachable_jointsl/attach</attach_topic>
+            <detach_topic>/detachable_jointsl/detach</detach_topic>
+            <output_topic>/detachable_jointsl/output</output_topic>
+            <grip_link>cylinder1_link</grip_link>
         </plugin>
-        <plugin name="gz::sim::systems::JointPositionController" filename="gz-sim-joint-position-controller-system">
-            <topic>can_gripper_joint_topic_2</topic>
-            <joint_name>can_gripper_joint_2</joint_name>
-            <p_gain>10</p_gain>
-            <i_gain>0.1</i_gain>
-            <d_gain>0.01</d_gain>
-            <i_max>1</i_max>
-            <i_min>-1</i_min>
-            <cmd_max>1000</cmd_max>
-            <cmd_min>-1000</cmd_min>
-        </plugin>
+        <plugin name="gripper_plugin_gz::DynamicDetachableJoint" filename="libgripper_plugin_gz.so">
+            <parent_link>col_gripper</parent_link>
+            <attach_topic>/detachable_jointsr/attach</attach_topic>
+            <detach_topic>/detachable_jointsr/detach</detach_topic>
+            <output_topic>/detachable_jointsr/output</output_topic>
+            <grip_link>cylinder1_link</grip_link>
+        </plugin> -->
     </gazebo>
 </robot>

File: src/shesnar/urdf/robot.urdf.xacro (robot description, xacro)
@@ -3,5 +3,4 @@
     <xacro:include filename="robot_core.xacro"/>
     <xacro:include filename="lidar.xacro"/>
-    <!-- <xacro:include filename="gripper.xacro"/> -->
     <xacro:include filename="robot_lifters.xacro"/>
     <!-- <xacro:include filename="sim_gripper_gz.xacro"/>  -->

File: src/shesnar/urdf/robot_lifters.xacro (robot description, xacro)
@@ -62,5 +62,5 @@
     </joint>
     <!-- Revolute Joint 1 (вращение банки 1) -->
-    <link name="can_rotator_1_link">
+    <!-- <link name="can_rotator_1_link">
         <visual>
             <geometry>
@@ -71,9 +71,9 @@
             </material>
         </visual>
-    </link>
-    <link name="can_rotator_1_cube">
+    </link> -->
+    <!-- <link name="can_rotator_1_cube">
         <visual>
             <geometry>
-                <box size="0.03 0.03 0.03"/>                      <!-- завхват банки №1 -->
+                <box size="0.03 0.03 0.03"/>                      завхват банки №1
             </geometry>
             <material name="blue">
@@ -89,15 +89,7 @@
         <child link="can_rotator_1_cube"/>
         <origin xyz="0.05 0 0.05" rpy="0 0 0"/>
-    </joint>
-    <joint name="can_rotator_1_joint" type="revolute">
-        <parent link="can_lift_link"/>
-        <child link="can_rotator_1_link"/>
-        <origin xyz="0 0.05 0" rpy="0 0 0"/>
-        <axis xyz="0 0 1"/>
-        <limit lower="-1.57" upper="1.57" effort="5" velocity="7.0"/>
-        <dynamics damping="0.1"/>
-    </joint>
+    </joint> -->
     <!-- Revolute Joint 2 (вращение банки 2) -->
-    <link name="can_rotator_2_link">
+    <!-- <link name="can_rotator_2_link">
         <visual>
             <geometry>
@@ -108,6 +100,6 @@
             </material>
         </visual>
-    </link>
-    <link name="can_rotator_2_cube">
+    </link> -->
+    <!-- <link name="can_rotator_2_cube">
         <visual>
             <geometry>
@@ -116,5 +108,5 @@
             <material name="blue">
                 <color rgba="0.0 0.0 1.0 1.0"/>
-            </material>                                                       <!-- завхват банки №2 -->
+            </material>                                                     завхват банки №2
         </visual>
         <xacro:inertial_box mass="0.1" x="0.05" y="0.05" z='0.05'>
@@ -126,13 +118,5 @@
         <child link="can_rotator_2_cube"/>
         <origin xyz="0.05 0 0.05" rpy="0 0 0"/>
-    </joint>
-    <joint name="can_rotator_2_joint" type="revolute">
-        <parent link="can_lift_link"/>
-        <child link="can_rotator_2_link"/>
-        <origin xyz="0 -0.05 0" rpy="0 0 0"/>
-        <axis xyz="0 0 -1"/>
-        <limit lower="-1.57" upper="1.57" effort="5" velocity="7.0"/>
-         <dynamics damping="0.1"/>
-    </joint>
+    </joint> -->
       <gazebo>
         <plugin name="gz::sim::systems::JointStatePublisher" filename="gz-sim-joint-state-publisher-system">
@@ -169,5 +153,5 @@
             <topic>can_rotator_1_topic</topic>
             <joint_name>can_rotator_1_joint</joint_name>
-            <p_gain>10</p_gain>
+            <p_gain>100</p_gain>
             <i_gain>0.1</i_gain>
             <d_gain>0.01</d_gain>
@@ -180,5 +164,5 @@
             <topic>can_rotator_2_topic</topic>
             <joint_name>can_rotator_2_joint</joint_name>
-            <p_gain>10</p_gain>
+            <p_gain>100</p_gain>
             <i_gain>0.1</i_gain>
             <d_gain>0.01</d_gain>

File: src/shesnar/urdf/sim_gripper_gz.xacro (robot description, xacro)
@@ -1,5 +1,5 @@
 <?xml version="1.0"?>
 <robot xmlns:xacro="http://www.ros.org/wiki/xacro">
-    <joint name="gripper_joint" type="prismatic">
+    <!-- <joint name="gripper_joint" type="prismatic">
         <parent link="body"/>
         <child link="col_gripper"/>
@@ -46,4 +46,5 @@
         </collision>
     </link>
+ -->
         <!-- <plugin name="gz::sim::systems::OdometryPublisher" filename="gz-sim-odometry-publisher-system">
             <odom_frame>odom</odom_frame>
@@ -55,23 +56,23 @@
     <gazebo>
         <plugin name="gripper_plugin_gz::DynamicDetachableJoint" filename="libgripper_plugin_gz.so">
-            <parent_link>col_gripper</parent_link>
+            <parent_link>can_gripper_1</parent_link>
             <attach_topic>/detachable_jointcl/attach</attach_topic>
             <detach_topic>/detachable_jointcl/detach</detach_topic>
             <output_topic>/detachable_jointcl/output</output_topic>
-            <!-- <grip_link>cylinder1_link</grip_link> -->
+            <grip_link>grip_link</grip_link>
         </plugin>
         <plugin name="gripper_plugin_gz::DynamicDetachableJoint" filename="libgripper_plugin_gz.so">
-            <parent_link>col_gripper</parent_link>
+            <parent_link>can_gripper_2</parent_link>
             <attach_topic>/detachable_jointcr/attach</attach_topic>
             <detach_topic>/detachable_jointcr/detach</detach_topic>
             <output_topic>/detachable_jointcr/output</output_topic>
-            <!-- <grip_link>cylinder1_link</grip_link> -->
+            <grip_link>grip_link</grip_link>
         </plugin>
-        <plugin name="gripper_plugin_gz::DynamicDetachableJoint" filename="libgripper_plugin_gz.so">
+        <!-- <plugin name="gripper_plugin_gz::DynamicDetachableJoint" filename="libgripper_plugin_gz.so">
             <parent_link>col_gripper</parent_link>
             <attach_topic>/detachable_jointsl/attach</attach_topic>
             <detach_topic>/detachable_jointsl/detach</detach_topic>
             <output_topic>/detachable_jointsl/output</output_topic>
-            <!-- <grip_link>cylinder1_link</grip_link> -->
+            <grip_link>cylinder1_link</grip_link>
         </plugin>
         <plugin name="gripper_plugin_gz::DynamicDetachableJoint" filename="libgripper_plugin_gz.so">
@@ -80,7 +81,6 @@
             <detach_topic>/detachable_jointsr/detach</detach_topic>
             <output_topic>/detachable_jointsr/output</output_topic>
-            <!-- <grip_link>cylinder1_link</grip_link> -->
+            <grip_link>cylinder1_link</grip_link>
         </plugin>
-<!--
         <plugin name="gz::sim::systems::DetachableJoint" filename="gz-sim-detachable-joint-system">
             <parent_link>col_gripper</parent_link>
@@ -114,6 +114,6 @@
             <detach_topic>/cylinder1/detach</detach_topic>
         </plugin> -->
-        <plugin name="gz::sim::systems::JointStatePublisher" filename="gz-sim-joint-state-publisher-system">
-            <!-- <topic>joint_states</topic>  -->
+        <!-- <plugin name="gz::sim::systems::JointStatePublisher" filename="gz-sim-joint-state-publisher-system">
+            <topic>joint_states</topic>
             <joint_name>gripper_joint</joint_name>
         </plugin>
@@ -128,5 +128,5 @@
             <cmd_max>1000</cmd_max>
             <cmd_min>-1000</cmd_min>
-        </plugin>
+        </plugin> -->
         <!-- <plugin name="gz::sim::systems::DetachableJoint">
         </plugin> -->
