Commit message: setup grippers

File: src/shesnar/urdf/can_gripper.xacro (robot description, xacro)
@@ -109,4 +109,112 @@
         <limit effort="1000.0" lower="0" upper="0.01" velocity="0.5"/>
     </joint>
+    <link name="can_gripper_sl">
+        <visual>
+            <origin xyz="0.0 0 0" rpy="0 0 -1.57" />
+            <geometry>
+                <box size="0.05 0.02 0.02"/>
+            </geometry>
+            <material name="blue">
+                <color rgba="0.0 0.0 1.0 1.0"/>
+            </material>
+        </visual>
+        <collision>
+            <origin xyz="0.0 0 0.0" rpy="0 0 -1.57" />
+            <geometry>
+                <box size="0.05 0.02 0.02"/>
+            </geometry>
+        </collision>
+        <xacro:inertial_box mass="0.01" x="0.05" y="0.02" z="0.02">
+            <origin xyz="0.0 0 0" rpy="0 0 0"/>
+        </xacro:inertial_box>
+    </link>
+    <joint name="can_gripper_joint_sl" type="prismatic">
+        <parent link="body"/>
+        <child link="can_gripper_sl"/>
+        <origin xyz="0.15 0.15 0.08" rpy="0 0 0"/>
+        <axis xyz="0 0 1"/>
+        <limit effort="1000.0" lower="0" upper="0.01" velocity="0.5"/>
+    </joint>
+    <link name="can_gripper_sr">
+        <visual>
+            <origin xyz="0.0 0 0" rpy="0 0 -1.57" />
+            <geometry>
+                <box size="0.05 0.02 0.02"/>
+            </geometry>
+            <material name="blue">
+                <color rgba="0.0 0.0 1.0 1.0"/>
+            </material>
+        </visual>
+        <collision>
+            <origin xyz="0.0 0 0.0" rpy="0 0 -1.57" />
+            <geometry>
+                <box size="0.05 0.02 0.02"/>
+            </geometry>
+        </collision>
+        <xacro:inertial_box mass="0.01" x="0.05" y="0.02" z="0.02">
+            <origin xyz="0.0 0 0" rpy="0 0 0"/>
+        </xacro:inertial_box>
+    </link>
+    <joint name="can_gripper_joint_sr" type="prismatic">
+        <parent link="body"/>
+        <child link="can_gripper_sr"/>
+        <origin xyz="0.15 -0.15 0.08" rpy="0 0 0"/>
+        <axis xyz="0 0 1"/>
+        <limit effort="1000.0" lower="0" upper="0.01" velocity="0.5"/>
+    </joint>
+    <link name="can_gripper_sl">
+        <visual>
+            <origin xyz="0.0 0 0" rpy="0 0 -1.57" />
+            <geometry>
+                <box size="0.05 0.02 0.02"/>
+            </geometry>
+            <material name="blue">
+                <color rgba="0.0 0.0 1.0 1.0"/>
+            </material>
+        </visual>
+        <collision>
+            <origin xyz="0.0 0 0.0" rpy="0 0 -1.57" />
+            <geometry>
+                <box size="0.05 0.02 0.02"/>
+            </geometry>
+        </collision>
+        <xacro:inertial_box mass="0.01" x="0.05" y="0.02" z="0.02">
+            <origin xyz="0.0 0 0" rpy="0 0 0"/>
+        </xacro:inertial_box>
+    </link>
+    <joint name="can_gripper_joint_sl" type="prismatic">
+        <parent link="body"/>
+        <child link="can_gripper_sl"/>
+        <origin xyz="0.15 0.15 0.08" rpy="0 0 0"/>
+        <axis xyz="0 0 1"/>
+        <limit effort="1000.0" lower="0" upper="0.01" velocity="0.5"/>
+    </joint>
+    <link name="can_gripper_sr">
+        <visual>
+            <origin xyz="0.0 0 0" rpy="0 0 -1.57" />
+            <geometry>
+                <box size="0.05 0.02 0.02"/>
+            </geometry>
+            <material name="blue">
+                <color rgba="0.0 0.0 1.0 1.0"/>
+            </material>
+        </visual>
+        <collision>
+            <origin xyz="0.0 0 0.0" rpy="0 0 -1.57" />
+            <geometry>
+                <box size="0.05 0.02 0.02"/>
+            </geometry>
+        </collision>
+        <xacro:inertial_box mass="0.01" x="0.05" y="0.02" z="0.02">
+            <origin xyz="0.0 0 0" rpy="0 0 0"/>
+        </xacro:inertial_box>
+    </link>
+    <joint name="can_gripper_joint_sr" type="prismatic">
+        <parent link="body"/>
+        <child link="can_gripper_sr"/>
+        <origin xyz="0.15 -0.15 0.08" rpy="0 0 0"/>
+        <axis xyz="0 0 1"/>
+        <limit effort="1000.0" lower="0" upper="0.01" velocity="0.5"/>
+    </joint>
     <gazebo>
         <plugin name="gripper_plugin_gz::DynamicDetachableJoint" filename="libgripper_plugin_gz.so">
@@ -146,10 +254,10 @@
         </plugin>
         <plugin name="gripper_plugin_gz::DynamicDetachableJoint" filename="libgripper_plugin_gz.so">
-            <parent_link>col_gripper</parent_link>
+            <parent_link>can_gripper_sr</parent_link>
             <attach_topic>/detachable_jointsr/attach</attach_topic>
             <detach_topic>/detachable_jointsr/detach</detach_topic>
             <output_topic>/detachable_jointsr/output</output_topic>
-            <grip_link>cylinder1_link</grip_link>
-        </plugin> -->
+            <grip_link>grip_link</grip_link>
+        </plugin>
     </gazebo>
 </robot>

File: src/shesnar/urdf/robot_lifters.xacro (robot description, xacro)
@@ -223,5 +223,5 @@
             <p_gain>100</p_gain>
             <i_gain>0.1</i_gain>
-            <d_gain>10.0</d_gain>
+            <d_gain>0.01</d_gain>
             <i_max>1</i_max>
             <i_min>-1</i_min>
@@ -231,5 +231,5 @@
         <plugin name="gz::sim::systems::JointPositionController" filename="gz-sim-joint-position-controller-system">
             <topic>can_rotator_1_topic</topic>
-            <joint_name>can_rotator_1_joint</joint_name>
+            <joint_name>can_gripper_joint_cr</joint_name>
             <p_gain>100</p_gain>
             <i_gain>0.1</i_gain>
@@ -242,5 +242,5 @@
         <plugin name="gz::sim::systems::JointPositionController" filename="gz-sim-joint-position-controller-system">
             <topic>can_rotator_2_topic</topic>
-            <joint_name>can_rotator_2_joint</joint_name>
+            <joint_name>can_gripper_joint_cl</joint_name>
             <p_gain>100</p_gain>
             <i_gain>0.1</i_gain>

Commit message: setup grippers

File: src/shesnar/urdf/can_gripper.xacro (robot description, xacro)
@@ -1,5 +1,5 @@
 <?xml version="1.0"?>
 <robot xmlns:xacro="http://www.ros.org/wiki/xacro">
-    <link name="can_gripper_1">
+    <link name="can_gripper_cr">
         <visual>
             <origin xyz="0.0 0 0.0" rpy="0 0 1.57" />
@@ -21,12 +21,12 @@
         </xacro:inertial_box>
     </link>
-    <joint name="can_gripper_joint_1" type="prismatic">
+    <joint name="can_gripper_joint_cr" type="prismatic">
         <parent link="can_lift_link"/>
-        <child link="can_gripper_1"/>
+        <child link="can_gripper_cr"/>
         <origin xyz="0.05 -0.05 0.05" rpy="0 0 0"/>
         <axis xyz="1 0 0"/>
         <limit effort="1000.0" lower="0" upper="0.1" velocity="0.5"/>
     </joint>
-    <link name="can_gripper_2">
+    <link name="can_gripper_cl">
         <visual>
             <origin xyz="0.0 0 0" rpy="0 0 -1.57" />
@@ -48,14 +48,68 @@
         </xacro:inertial_box>
     </link>
-    <joint name="can_gripper_joint_2" type="prismatic">
+    <joint name="can_gripper_joint_cl" type="prismatic">
         <parent link="can_lift_link"/>
-        <child link="can_gripper_2"/>
+        <child link="can_gripper_cl"/>
         <origin xyz="0.05 0.05 0.05" rpy="0 0 0"/>
         <axis xyz="1 0 0"/>
         <limit effort="1000.0" lower="0" upper="0.1" velocity="0.5"/>
     </joint>
+    <link name="can_gripper_sl">
+        <visual>
+            <origin xyz="0.0 0 0" rpy="0 0 -1.57" />
+            <geometry>
+                <box size="0.05 0.02 0.02"/>
+            </geometry>
+            <material name="blue">
+                <color rgba="0.0 0.0 1.0 1.0"/>
+            </material>
+        </visual>
+        <collision>
+            <origin xyz="0.0 0 0.0" rpy="0 0 -1.57" />
+            <geometry>
+                <box size="0.05 0.02 0.02"/>
+            </geometry>
+        </collision>
+        <xacro:inertial_box mass="0.01" x="0.05" y="0.02" z="0.02">
+            <origin xyz="0.0 0 0" rpy="0 0 0"/>
+        </xacro:inertial_box>
+    </link>
+    <joint name="can_gripper_joint_sl" type="prismatic">
+        <parent link="body"/>
+        <child link="can_gripper_sl"/>
+        <origin xyz="0.15 0.15 0.08" rpy="0 0 0"/>
+        <axis xyz="0 0 1"/>
+        <limit effort="1000.0" lower="0" upper="0.01" velocity="0.5"/>
+    </joint>
+    <link name="can_gripper_sr">
+        <visual>
+            <origin xyz="0.0 0 0" rpy="0 0 -1.57" />
+            <geometry>
+                <box size="0.05 0.02 0.02"/>
+            </geometry>
+            <material name="blue">
+                <color rgba="0.0 0.0 1.0 1.0"/>
+            </material>
+        </visual>
+        <collision>
+            <origin xyz="0.0 0 0.0" rpy="0 0 -1.57" />
+            <geometry>
+                <box size="0.05 0.02 0.02"/>
+            </geometry>
+        </collision>
+        <xacro:inertial_box mass="0.01" x="0.05" y="0.02" z="0.02">
+            <origin xyz="0.0 0 0" rpy="0 0 0"/>
+        </xacro:inertial_box>
+    </link>
+    <joint name="can_gripper_joint_sr" type="prismatic">
+        <parent link="body"/>
+        <child link="can_gripper_sr"/>
+        <origin xyz="0.15 -0.15 0.08" rpy="0 0 0"/>
+        <axis xyz="0 0 1"/>
+        <limit effort="1000.0" lower="0" upper="0.01" velocity="0.5"/>
+    </joint>
     <gazebo>
         <plugin name="gripper_plugin_gz::DynamicDetachableJoint" filename="libgripper_plugin_gz.so">
-            <parent_link>can_gripper_1</parent_link>
+            <parent_link>can_gripper_cl</parent_link>
             <attach_topic>/detachable_jointcl/attach</attach_topic>
             <detach_topic>/detachable_jointcl/detach</detach_topic>
@@ -64,5 +118,5 @@
         </plugin>
         <plugin name="gripper_plugin_gz::DynamicDetachableJoint" filename="libgripper_plugin_gz.so">
-            <parent_link>can_gripper_2</parent_link>
+            <parent_link>can_gripper_cr</parent_link>
             <attach_topic>/detachable_jointcr/attach</attach_topic>
             <detach_topic>/detachable_jointcr/detach</detach_topic>
@@ -70,18 +124,18 @@
             <grip_link>grip_link</grip_link>
         </plugin>
-        <!-- <plugin name="gripper_plugin_gz::DynamicDetachableJoint" filename="libgripper_plugin_gz.so">
-            <parent_link>col_gripper</parent_link>
+        <plugin name="gripper_plugin_gz::DynamicDetachableJoint" filename="libgripper_plugin_gz.so">
+            <parent_link>can_gripper_sl</parent_link>
             <attach_topic>/detachable_jointsl/attach</attach_topic>
             <detach_topic>/detachable_jointsl/detach</detach_topic>
             <output_topic>/detachable_jointsl/output</output_topic>
-            <grip_link>cylinder1_link</grip_link>
+            <grip_link>grip_link</grip_link>
         </plugin>
         <plugin name="gripper_plugin_gz::DynamicDetachableJoint" filename="libgripper_plugin_gz.so">
-            <parent_link>col_gripper</parent_link>
+            <parent_link>can_gripper_sr</parent_link>
             <attach_topic>/detachable_jointsr/attach</attach_topic>
             <detach_topic>/detachable_jointsr/detach</detach_topic>
             <output_topic>/detachable_jointsr/output</output_topic>
-            <grip_link>cylinder1_link</grip_link>
-        </plugin> -->
+            <grip_link>grip_link</grip_link>
+        </plugin>
     </gazebo>
 </robot>

File: src/shesnar/urdf/robot_lifters.xacro (robot description, xacro)
@@ -59,5 +59,5 @@
         <origin xyz="0.1 0.0 0.028" rpy="0 0 0"/>
         <axis xyz="0 0 1"/>
-        <limit effort="1000.0" lower="0" upper="0.11" velocity="0.5"/>
+        <limit effort="1000.0" lower="0" upper="0.2" velocity="0.5"/>
     </joint>
     <!-- Revolute Joint 1 (вращение банки 1) -->
@@ -144,5 +144,5 @@
             <p_gain>100</p_gain>
             <i_gain>0.1</i_gain>
-            <d_gain>10.0</d_gain>
+            <d_gain>0.01</d_gain>
             <i_max>1</i_max>
             <i_min>-1</i_min>
@@ -152,5 +152,5 @@
         <plugin name="gz::sim::systems::JointPositionController" filename="gz-sim-joint-position-controller-system">
             <topic>can_rotator_1_topic</topic>
-            <joint_name>can_rotator_1_joint</joint_name>
+            <joint_name>can_gripper_joint_cr</joint_name>
             <p_gain>100</p_gain>
             <i_gain>0.1</i_gain>
@@ -163,5 +163,5 @@
         <plugin name="gz::sim::systems::JointPositionController" filename="gz-sim-joint-position-controller-system">
             <topic>can_rotator_2_topic</topic>
-            <joint_name>can_rotator_2_joint</joint_name>
+            <joint_name>can_gripper_joint_cl</joint_name>
             <p_gain>100</p_gain>
             <i_gain>0.1</i_gain>

Commit message: new body

File: src/shesnar/urdf/can_gripper.xacro (robot description, xacro)
@@ -108,4 +108,6 @@
         <axis xyz="0 0 1"/>
         <limit effort="1000.0" lower="0" upper="0.01" velocity="0.5"/>
+=======
+>>>>>>> 97f6fc5 (new body)
     </joint>
     <link name="can_gripper_sl">
@@ -132,5 +134,5 @@
         <parent link="body"/>
         <child link="can_gripper_sl"/>
-        <origin xyz="0.15 0.15 0.08" rpy="0 0 0"/>
+        <origin xyz="0.13 0.15 0.08" rpy="0 0 0"/>
         <axis xyz="0 0 1"/>
         <limit effort="1000.0" lower="0" upper="0.01" velocity="0.5"/>
@@ -159,59 +161,5 @@
         <parent link="body"/>
         <child link="can_gripper_sr"/>
-        <origin xyz="0.15 -0.15 0.08" rpy="0 0 0"/>
-        <axis xyz="0 0 1"/>
-        <limit effort="1000.0" lower="0" upper="0.01" velocity="0.5"/>
-    </joint>
-    <link name="can_gripper_sl">
-        <visual>
-            <origin xyz="0.0 0 0" rpy="0 0 -1.57" />
-            <geometry>
-                <box size="0.05 0.02 0.02"/>
-            </geometry>
-            <material name="blue">
-                <color rgba="0.0 0.0 1.0 1.0"/>
-            </material>
-        </visual>
-        <collision>
-            <origin xyz="0.0 0 0.0" rpy="0 0 -1.57" />
-            <geometry>
-                <box size="0.05 0.02 0.02"/>
-            </geometry>
-        </collision>
-        <xacro:inertial_box mass="0.01" x="0.05" y="0.02" z="0.02">
-            <origin xyz="0.0 0 0" rpy="0 0 0"/>
-        </xacro:inertial_box>
-    </link>
-    <joint name="can_gripper_joint_sl" type="prismatic">
-        <parent link="body"/>
-        <child link="can_gripper_sl"/>
-        <origin xyz="0.15 0.15 0.08" rpy="0 0 0"/>
-        <axis xyz="0 0 1"/>
-        <limit effort="1000.0" lower="0" upper="0.01" velocity="0.5"/>
-    </joint>
-    <link name="can_gripper_sr">
-        <visual>
-            <origin xyz="0.0 0 0" rpy="0 0 -1.57" />
-            <geometry>
-                <box size="0.05 0.02 0.02"/>
-            </geometry>
-            <material name="blue">
-                <color rgba="0.0 0.0 1.0 1.0"/>
-            </material>
-        </visual>
-        <collision>
-            <origin xyz="0.0 0 0.0" rpy="0 0 -1.57" />
-            <geometry>
-                <box size="0.05 0.02 0.02"/>
-            </geometry>
-        </collision>
-        <xacro:inertial_box mass="0.01" x="0.05" y="0.02" z="0.02">
-            <origin xyz="0.0 0 0" rpy="0 0 0"/>
-        </xacro:inertial_box>
-    </link>
-    <joint name="can_gripper_joint_sr" type="prismatic">
-        <parent link="body"/>
-        <child link="can_gripper_sr"/>
-        <origin xyz="0.15 -0.15 0.08" rpy="0 0 0"/>
+        <origin xyz="0.13 -0.15 0.08" rpy="0 0 0"/>
         <axis xyz="0 0 1"/>
         <limit effort="1000.0" lower="0" upper="0.01" velocity="0.5"/>
@@ -254,10 +202,10 @@
         </plugin>
         <plugin name="gripper_plugin_gz::DynamicDetachableJoint" filename="libgripper_plugin_gz.so">
-            <parent_link>can_gripper_sr</parent_link>
+            <parent_link>col_gripper</parent_link>
             <attach_topic>/detachable_jointsr/attach</attach_topic>
             <detach_topic>/detachable_jointsr/detach</detach_topic>
             <output_topic>/detachable_jointsr/output</output_topic>
-            <grip_link>grip_link</grip_link>
-        </plugin>
+            <grip_link>cylinder1_link</grip_link>
+        </plugin> -->
     </gazebo>
 </robot>

Commit message: new body

File: src/shesnar/urdf/can_gripper.xacro (robot description, xacro)
@@ -24,7 +24,7 @@
         <parent link="can_lift_link"/>
         <child link="can_gripper_cr"/>
-        <origin xyz="0.05 -0.05 0.05" rpy="0 0 0"/>
+        <origin xyz="0.09 -0.05 0.0" rpy="0 0 0"/>
         <axis xyz="1 0 0"/>
-        <limit effort="1000.0" lower="0" upper="0.1" velocity="0.5"/>
+        <limit effort="1000.0" lower="0" upper="0.04" velocity="0.5"/>
     </joint>
     <link name="can_gripper_cl">
@@ -51,7 +51,7 @@
         <parent link="can_lift_link"/>
         <child link="can_gripper_cl"/>
-        <origin xyz="0.05 0.05 0.05" rpy="0 0 0"/>
+        <origin xyz="0.09 0.05 0.0" rpy="0 0 0"/>
         <axis xyz="1 0 0"/>
-        <limit effort="1000.0" lower="0" upper="0.1" velocity="0.5"/>
+        <limit effort="1000.0" lower="0" upper="0.04" velocity="0.5"/>
     </joint>
     <link name="can_gripper_sl">
@@ -78,5 +78,5 @@
         <parent link="body"/>
         <child link="can_gripper_sl"/>
-        <origin xyz="0.15 0.15 0.08" rpy="0 0 0"/>
+        <origin xyz="0.13 0.15 0.08" rpy="0 0 0"/>
         <axis xyz="0 0 1"/>
         <limit effort="1000.0" lower="0" upper="0.01" velocity="0.5"/>
@@ -105,5 +105,5 @@
         <parent link="body"/>
         <child link="can_gripper_sr"/>
-        <origin xyz="0.15 -0.15 0.08" rpy="0 0 0"/>
+        <origin xyz="0.13 -0.15 0.08" rpy="0 0 0"/>
         <axis xyz="0 0 1"/>
         <limit effort="1000.0" lower="0" upper="0.01" velocity="0.5"/>

File: src/shesnar/urdf/robot_core.xacro (robot description, xacro)
@@ -36,5 +36,5 @@
             <origin xyz="0.1 -0.18 0" rpy="1.57 0 1.57" />
             <geometry>
-                <mesh scale="0.1 0.1 0.1" rpy="0 0 1.04" filename="file://$(find shesnar)/meshes/body.obj"/>
+                <mesh scale="0.1 0.1 0.1" rpy="0 0 1.04" filename="file://$(find shesnar)/meshes/body2.obj"/>
             <!-- <cylinder radius="0.20" length="0.12"/> -->
             </geometry>
@@ -46,5 +46,5 @@
             <origin xyz="0.1 -0.18 0" rpy="1.57 0 1.57" />
             <geometry>
-                 <mesh scale="0.1 0.1 0.1" rpy="0 0 1.04" filename="file://$(find shesnar)/meshes/body_collision.obj"/>
+                 <mesh scale="0.1 0.1 0.1" rpy="0 0 1.04" filename="file://$(find shesnar)/meshes/body2.obj"/>
                 <!-- <cylinder radius="0.20" length="0.12"/> -->
             </geometry>

File: src/shesnar/urdf/robot_lifters.xacro (robot description, xacro)
@@ -57,5 +57,5 @@
         <parent link="body"/>
         <child link="can_lift_link"/>
-        <origin xyz="0.1 0.0 0.028" rpy="0 0 0"/>
+        <origin xyz="0.0 0.0 0.07" rpy="0 0 0"/>
         <axis xyz="0 0 1"/>
         <limit effort="1000.0" lower="0" upper="0.2" velocity="0.5"/>
