Commit message: Fixed lifters work under load

File: src/shesnar/urdf/can_gripper.xacro (robot description, xacro)
@@ -26,5 +26,5 @@
         <origin xyz="0.09 -0.05 0.0" rpy="0 0 0"/>
         <axis xyz="1 0 0"/>
-        <limit effort="1000.0" lower="0" upper="0.04" velocity="0.5"/>
+        <limit effort="30.0" lower="0" upper="0.04" velocity="0.5"/>
     </joint>
     <link name="can_gripper_cl">
@@ -53,5 +53,5 @@
         <origin xyz="0.09 0.05 0.0" rpy="0 0 0"/>
         <axis xyz="1 0 0"/>
-        <limit effort="1000.0" lower="0" upper="0.04" velocity="0.5"/>
+        <limit effort="30.0" lower="0" upper="0.04" velocity="0.5"/>
     </joint>
     <link name="can_gripper_sl">
@@ -80,5 +80,5 @@
         <origin xyz="0.13 0.15 0.08" rpy="0 0 0"/>
         <axis xyz="0 0 1"/>
-        <limit effort="1000.0" lower="0" upper="0.01" velocity="0.5"/>
+        <limit effort="30.0" lower="0" upper="0.01" velocity="0.5"/>
     </joint>
     <link name="can_gripper_sr">
@@ -107,4 +107,5 @@
         <origin xyz="0.13 -0.15 0.08" rpy="0 0 0"/>
         <axis xyz="0 0 1"/>
+<<<<<<< HEAD
         <limit effort="1000.0" lower="0" upper="0.01" velocity="0.5"/>
 =======
@@ -164,4 +165,7 @@
         <axis xyz="0 0 1"/>
         <limit effort="1000.0" lower="0" upper="0.01" velocity="0.5"/>
+=======
+        <limit effort="30.0" lower="0" upper="0.01" velocity="0.5"/>
+>>>>>>> dbd8180 (Fixed lifters work under load)
     </joint>
     <gazebo>

File: src/shesnar/urdf/robot_lifters.xacro (robot description, xacro)
@@ -38,5 +38,5 @@
         <origin xyz="0 0 0.14" rpy="0 0 0"/>
         <axis xyz="0 0 1"/>
-        <limit lower="0" upper="0.11" effort="1000.0" velocity="0.5"/>
+        <limit lower="0" upper="0.11" effort="30.0" velocity="0.5"/>
     </joint>
     <!-- Prismatic Joint 2 (подъём банок) -->
@@ -59,5 +59,5 @@
         <origin xyz="0.0 0.0 0.07" rpy="0 0 0"/>
         <axis xyz="0 0 1"/>
-        <limit effort="1000.0" lower="0" upper="0.2" velocity="0.5"/>
+        <limit effort="30.0" lower="0" upper="0.2" velocity="0.5"/>
     </joint>
     <!-- Revolute Joint 1 (вращение банки 1) -->
@@ -209,28 +209,28 @@
             <joint_name>board_lift_joint</joint_name>
             <!-- <joint_index>1</joint_index> -->
-            <p_gain>100</p_gain>
-            <i_gain>0.1</i_gain>
+            <p_gain>2000.0</p_gain>
+            <i_gain>0.1</i_gain>
+            <d_gain>20.0</d_gain>
+            <i_max>1</i_max>
+            <i_min>-1</i_min>
+            <cmd_max>20000</cmd_max>
+            <cmd_min>-20000</cmd_min>
+        </plugin>
+        <plugin name="gz::sim::systems::JointPositionController" filename="gz-sim-joint-position-controller-system">
+            <topic>can_lift_topic</topic>
+            <joint_name>can_lift_joint</joint_name>
+            <!-- <joint_index>1</joint_index> -->
+            <p_gain>200</p_gain>
+            <i_gain>1.0</i_gain>
             <d_gain>10.0</d_gain>
             <i_max>1</i_max>
             <i_min>-1</i_min>
-            <cmd_max>50000</cmd_max>
-            <cmd_min>-50000</cmd_min>
-        </plugin>
-        <plugin name="gz::sim::systems::JointPositionController" filename="gz-sim-joint-position-controller-system">
-            <topic>can_lift_topic</topic>
-            <joint_name>can_lift_joint</joint_name>
-            <!-- <joint_index>1</joint_index> -->
-            <p_gain>100</p_gain>
-            <i_gain>0.1</i_gain>
-            <d_gain>0.01</d_gain>
-            <i_max>1</i_max>
-            <i_min>-1</i_min>
-            <cmd_max>50000</cmd_max>
-            <cmd_min>-50000</cmd_min>
+            <cmd_max>20000</cmd_max>
+            <cmd_min>-20000</cmd_min>
         </plugin>
         <plugin name="gz::sim::systems::JointPositionController" filename="gz-sim-joint-position-controller-system">
             <topic>can_rotator_1_topic</topic>
             <joint_name>can_gripper_joint_cr</joint_name>
-            <p_gain>100</p_gain>
+            <p_gain>10</p_gain>
             <i_gain>0.1</i_gain>
             <d_gain>0.01</d_gain>
@@ -243,5 +243,5 @@
             <topic>can_rotator_2_topic</topic>
             <joint_name>can_gripper_joint_cl</joint_name>
-            <p_gain>100</p_gain>
+            <p_gain>10</p_gain>
             <i_gain>0.1</i_gain>
             <d_gain>0.01</d_gain>

Commit message: Fixed lifters work under load

File: src/shesnar/urdf/can_gripper.xacro (robot description, xacro)
@@ -26,5 +26,5 @@
         <origin xyz="0.09 -0.05 0.0" rpy="0 0 0"/>
         <axis xyz="1 0 0"/>
-        <limit effort="1000.0" lower="0" upper="0.04" velocity="0.5"/>
+        <limit effort="30.0" lower="0" upper="0.04" velocity="0.5"/>
     </joint>
     <link name="can_gripper_cl">
@@ -53,5 +53,5 @@
         <origin xyz="0.09 0.05 0.0" rpy="0 0 0"/>
         <axis xyz="1 0 0"/>
-        <limit effort="1000.0" lower="0" upper="0.04" velocity="0.5"/>
+        <limit effort="30.0" lower="0" upper="0.04" velocity="0.5"/>
     </joint>
     <link name="can_gripper_sl">
@@ -80,5 +80,5 @@
         <origin xyz="0.13 0.15 0.08" rpy="0 0 0"/>
         <axis xyz="0 0 1"/>
-        <limit effort="1000.0" lower="0" upper="0.01" velocity="0.5"/>
+        <limit effort="30.0" lower="0" upper="0.01" velocity="0.5"/>
     </joint>
     <link name="can_gripper_sr">
@@ -107,5 +107,5 @@
         <origin xyz="0.13 -0.15 0.08" rpy="0 0 0"/>
         <axis xyz="0 0 1"/>
-        <limit effort="1000.0" lower="0" upper="0.01" velocity="0.5"/>
+        <limit effort="30.0" lower="0" upper="0.01" velocity="0.5"/>
     </joint>
     <gazebo>

File: src/shesnar/urdf/robot_lifters.xacro (robot description, xacro)
@@ -38,5 +38,5 @@
         <origin xyz="0 0 0.14" rpy="0 0 0"/>
         <axis xyz="0 0 1"/>
-        <limit lower="0" upper="0.11" effort="1000.0" velocity="0.5"/>
+        <limit lower="0" upper="0.11" effort="30.0" velocity="0.5"/>
     </joint>
     <!-- Prismatic Joint 2 (подъём банок) -->
@@ -59,5 +59,5 @@
         <origin xyz="0.0 0.0 0.07" rpy="0 0 0"/>
         <axis xyz="0 0 1"/>
-        <limit effort="1000.0" lower="0" upper="0.2" velocity="0.5"/>
+        <limit effort="30.0" lower="0" upper="0.2" velocity="0.5"/>
     </joint>
     <!-- Revolute Joint 1 (вращение банки 1) -->
@@ -130,11 +130,11 @@
             <joint_name>board_lift_joint</joint_name>
             <!-- <joint_index>1</joint_index> -->
-            <p_gain>100</p_gain>
+            <p_gain>2000.0</p_gain>
             <i_gain>0.1</i_gain>
-            <d_gain>10.0</d_gain>
+            <d_gain>20.0</d_gain>
             <i_max>1</i_max>
             <i_min>-1</i_min>
-            <cmd_max>50000</cmd_max>
-            <cmd_min>-50000</cmd_min>
+            <cmd_max>20000</cmd_max>
+            <cmd_min>-20000</cmd_min>
         </plugin>
         <plugin name="gz::sim::systems::JointPositionController" filename="gz-sim-joint-position-controller-system">
@@ -142,16 +142,16 @@
             <joint_name>can_lift_joint</joint_name>
             <!-- <joint_index>1</joint_index> -->
-            <p_gain>100</p_gain>
-            <i_gain>0.1</i_gain>
-            <d_gain>0.01</d_gain>
+            <p_gain>200</p_gain>
+            <i_gain>1.0</i_gain>
+            <d_gain>10.0</d_gain>
             <i_max>1</i_max>
             <i_min>-1</i_min>
-            <cmd_max>50000</cmd_max>
-            <cmd_min>-50000</cmd_min>
+            <cmd_max>20000</cmd_max>
+            <cmd_min>-20000</cmd_min>
         </plugin>
         <plugin name="gz::sim::systems::JointPositionController" filename="gz-sim-joint-position-controller-system">
             <topic>can_rotator_1_topic</topic>
             <joint_name>can_gripper_joint_cr</joint_name>
-            <p_gain>100</p_gain>
+            <p_gain>10</p_gain>
             <i_gain>0.1</i_gain>
             <d_gain>0.01</d_gain>
@@ -164,5 +164,5 @@
             <topic>can_rotator_2_topic</topic>
             <joint_name>can_gripper_joint_cl</joint_name>
-            <p_gain>100</p_gain>
+            <p_gain>10</p_gain>
             <i_gain>0.1</i_gain>
             <d_gain>0.01</d_gain>

Commit message: setup_move

File: src/shesnar/urdf/can_gripper.xacro (robot description, xacro)
@@ -107,65 +107,5 @@
         <origin xyz="0.13 -0.15 0.08" rpy="0 0 0"/>
         <axis xyz="0 0 1"/>
-<<<<<<< HEAD
-        <limit effort="1000.0" lower="0" upper="0.01" velocity="0.5"/>
-=======
->>>>>>> 97f6fc5 (new body)
-    </joint>
-    <link name="can_gripper_sl">
-        <visual>
-            <origin xyz="0.0 0 0" rpy="0 0 -1.57" />
-            <geometry>
-                <box size="0.05 0.02 0.02"/>
-            </geometry>
-            <material name="blue">
-                <color rgba="0.0 0.0 1.0 1.0"/>
-            </material>
-        </visual>
-        <collision>
-            <origin xyz="0.0 0 0.0" rpy="0 0 -1.57" />
-            <geometry>
-                <box size="0.05 0.02 0.02"/>
-            </geometry>
-        </collision>
-        <xacro:inertial_box mass="0.01" x="0.05" y="0.02" z="0.02">
-            <origin xyz="0.0 0 0" rpy="0 0 0"/>
-        </xacro:inertial_box>
-    </link>
-    <joint name="can_gripper_joint_sl" type="prismatic">
-        <parent link="body"/>
-        <child link="can_gripper_sl"/>
-        <origin xyz="0.13 0.15 0.08" rpy="0 0 0"/>
-        <axis xyz="0 0 1"/>
-        <limit effort="1000.0" lower="0" upper="0.01" velocity="0.5"/>
-    </joint>
-    <link name="can_gripper_sr">
-        <visual>
-            <origin xyz="0.0 0 0" rpy="0 0 -1.57" />
-            <geometry>
-                <box size="0.05 0.02 0.02"/>
-            </geometry>
-            <material name="blue">
-                <color rgba="0.0 0.0 1.0 1.0"/>
-            </material>
-        </visual>
-        <collision>
-            <origin xyz="0.0 0 0.0" rpy="0 0 -1.57" />
-            <geometry>
-                <box size="0.05 0.02 0.02"/>
-            </geometry>
-        </collision>
-        <xacro:inertial_box mass="0.01" x="0.05" y="0.02" z="0.02">
-            <origin xyz="0.0 0 0" rpy="0 0 0"/>
-        </xacro:inertial_box>
-    </link>
-    <joint name="can_gripper_joint_sr" type="prismatic">
-        <parent link="body"/>
-        <child link="can_gripper_sr"/>
-        <origin xyz="0.13 -0.15 0.08" rpy="0 0 0"/>
-        <axis xyz="0 0 1"/>
-        <limit effort="1000.0" lower="0" upper="0.01" velocity="0.5"/>
-=======
         <limit effort="30.0" lower="0" upper="0.01" velocity="0.5"/>
->>>>>>> dbd8180 (Fixed lifters work under load)
     </joint>
     <gazebo>
@@ -205,11 +145,4 @@
             <grip_link>grip_link</grip_link>
         </plugin>
-        <plugin name="gripper_plugin_gz::DynamicDetachableJoint" filename="libgripper_plugin_gz.so">
-            <parent_link>col_gripper</parent_link>
-            <attach_topic>/detachable_jointsr/attach</attach_topic>
-            <detach_topic>/detachable_jointsr/detach</detach_topic>
-            <output_topic>/detachable_jointsr/output</output_topic>
-            <grip_link>cylinder1_link</grip_link>
-        </plugin> -->
     </gazebo>
 </robot>

File: src/shesnar/urdf/robot_lifters.xacro (robot description, xacro)
@@ -38,5 +38,5 @@
         <origin xyz="0 0 0.14" rpy="0 0 0"/>
         <axis xyz="0 0 1"/>
-        <limit lower="0" upper="0.11" effort="30.0" velocity="0.5"/>
+        <limit lower="0" upper="0.18" effort="30.0" velocity="0.5"/>
     </joint>
     <!-- Prismatic Joint 2 (подъём банок) -->
@@ -90,18 +90,4 @@
         <origin xyz="0.05 0 0.05" rpy="0 0 0"/>
     </joint> -->
-<<<<<<< HEAD
-<<<<<<< HEAD
-=======
-    <joint name="can_rotator_1_joint" type="revolute">
-        <parent link="can_lift_link"/>
-        <child link="can_rotator_1_link"/>
-        <origin xyz="0 0.05 0" rpy="0 0 0"/>
-        <axis xyz="0 0 1"/>
-        <limit lower="-1.57" upper="1.57" effort="5" velocity="7.0"/>
-        <dynamics damping="0.1"/>
-    </joint>
->>>>>>> b3c9261 (Added lifters_control)
-=======
->>>>>>> f41de3b (merge grip and art urdf)
     <!-- Revolute Joint 2 (вращение банки 2) -->
     <!-- <link name="can_rotator_2_link">
@@ -122,13 +108,5 @@
             <material name="blue">
                 <color rgba="0.0 0.0 1.0 1.0"/>
-<<<<<<< HEAD
-<<<<<<< HEAD
             </material>                                                     завхват банки №2
-=======
-            </material>                                                       <!-- завхват банки №2 -->
->>>>>>> b3c9261 (Added lifters_control)
-=======
-            </material>                                                     завхват банки №2
->>>>>>> f41de3b (merge grip and art urdf)
         </visual>
         <xacro:inertial_box mass="0.1" x="0.05" y="0.05" z='0.05'>
@@ -141,61 +119,4 @@
         <origin xyz="0.05 0 0.05" rpy="0 0 0"/>
     </joint> -->
-<<<<<<< HEAD
-      <gazebo>
-        <plugin name="gz::sim::systems::JointStatePublisher" filename="gz-sim-joint-state-publisher-system">
-            <!-- <joint_name>board_lift_joint</joint_name>
-            <joint_name>can_lift_joint</joint_name>
-            <joint_name>can_rotator_1_joint</joint_name>
-            <joint_name>can_rotator_2_joint</joint_name> -->
-        </plugin>
-        <plugin name="gz::sim::systems::JointPositionController" filename="gz-sim-joint-position-controller-system">
-            <topic>board_lift_topic</topic>
-            <joint_name>board_lift_joint</joint_name>
-            <!-- <joint_index>1</joint_index> -->
-            <p_gain>100</p_gain>
-            <i_gain>0.1</i_gain>
-            <d_gain>10.0</d_gain>
-            <i_max>1</i_max>
-            <i_min>-1</i_min>
-            <cmd_max>50000</cmd_max>
-            <cmd_min>-50000</cmd_min>
-        </plugin>
-        <plugin name="gz::sim::systems::JointPositionController" filename="gz-sim-joint-position-controller-system">
-            <topic>can_lift_topic</topic>
-            <joint_name>can_lift_joint</joint_name>
-            <!-- <joint_index>1</joint_index> -->
-            <p_gain>100</p_gain>
-            <i_gain>0.1</i_gain>
-            <d_gain>0.01</d_gain>
-            <i_max>1</i_max>
-            <i_min>-1</i_min>
-            <cmd_max>50000</cmd_max>
-            <cmd_min>-50000</cmd_min>
-        </plugin>
-        <plugin name="gz::sim::systems::JointPositionController" filename="gz-sim-joint-position-controller-system">
-            <topic>can_rotator_1_topic</topic>
-            <joint_name>can_gripper_joint_cr</joint_name>
-            <p_gain>100</p_gain>
-            <i_gain>0.1</i_gain>
-            <d_gain>0.01</d_gain>
-            <i_max>1</i_max>
-            <i_min>-1</i_min>
-            <cmd_max>1000</cmd_max>
-            <cmd_min>-1000</cmd_min>
-        </plugin>
-        <plugin name="gz::sim::systems::JointPositionController" filename="gz-sim-joint-position-controller-system">
-            <topic>can_rotator_2_topic</topic>
-            <joint_name>can_gripper_joint_cl</joint_name>
-            <p_gain>100</p_gain>
-            <i_gain>0.1</i_gain>
-            <d_gain>0.01</d_gain>
-            <i_max>1</i_max>
-            <i_min>-1</i_min>
-            <cmd_max>1000</cmd_max>
-            <cmd_min>-1000</cmd_min>
-        </plugin>
-    </gazebo>
-=======
->>>>>>> f41de3b (merge grip and art urdf)
       <gazebo>
         <plugin name="gz::sim::systems::JointStatePublisher" filename="gz-sim-joint-state-publisher-system">
@@ -233,8 +154,8 @@
             <joint_name>can_gripper_joint_cr</joint_name>
             <p_gain>10</p_gain>
-            <i_gain>0.1</i_gain>
+            <i_gain>0.7</i_gain>
             <d_gain>0.01</d_gain>
-            <i_max>1</i_max>
-            <i_min>-1</i_min>
+            <i_max>5</i_max>
+            <i_min>-5</i_min>
             <cmd_max>1000</cmd_max>
             <cmd_min>-1000</cmd_min>
@@ -244,8 +165,8 @@
             <joint_name>can_gripper_joint_cl</joint_name>
             <p_gain>10</p_gain>
-            <i_gain>0.1</i_gain>
+            <i_gain>0.7</i_gain>
             <d_gain>0.01</d_gain>
-            <i_max>1</i_max>
-            <i_min>-1</i_min>
+            <i_max>5</i_max>
+            <i_min>-5</i_min>
             <cmd_max>1000</cmd_max>
             <cmd_min>-1000</cmd_min>
