Commit message: normal robot camera added

File: src/shesnar/urdf/depth_camera.xacro (robot description, xacro)
@@ -4,10 +4,10 @@
         <parent link="body"/>
         <child link="camera_link"/>
-        <origin xyz="0 0 0.54"/>
+        <origin xyz="0.1 0 0.37" rpy="0 0.52 0"/>
     </joint>
     <link name="camera_link">
         <visual>
             <geometry>
-                <box size="0.1 0.3 0.3"/>
+                <box size="0.01 0.03 0.03"/>
             </geometry>
             <material name="red"/>
@@ -20,7 +20,6 @@
     </joint>
     <link name="camera_link_optical"></link>
-<!--
     <gazebo reference="camera_link">
-        <material>Gazebo/Black </material>
+        <material>Gazebo/Red </material>
         <sensor name="camera" type="camera">
             <pose> 0 0 0 0 0 0 </pose>
@@ -40,7 +39,7 @@
                 </clip>
             </camera>
-            <topic>camera/image_raw</topic>
+            <!-- <topic>camera/image_raw</topic> -->
             <gz_frame_id>camera_link</gz_frame_id>
         </sensor>
-    </gazebo> -->
+    </gazebo>
 </robot>

Commit message: depth_camera_added

File: src/shesnar/urdf/depth_camera.xacro (robot description, xacro)
@@ -4,5 +4,6 @@
         <parent link="body"/>
         <child link="camera_link"/>
-        <origin xyz="0.1 0 0.37" rpy="0 0.52 0"/>
+        <!-- <origin xyz="0.1 0 0.37" rpy="0 0.52 0"/> -->
+        <origin xyz="0.1 0 0.2" rpy="0 0 0"/>
     </joint>
     <link name="camera_link">
@@ -22,5 +23,5 @@
     <gazebo reference="camera_link">
         <material>Gazebo/Red </material>
-        <sensor name="camera" type="camera">
+        <sensor name="camera" type="depth_camera">
             <pose> 0 0 0 0 0 0 </pose>
             <visualize>true</visualize>

Commit message: depth camera new algorithm

File: src/shesnar/urdf/depth_camera.xacro (robot description, xacro)
@@ -2,8 +2,9 @@
 <robot xmlns:xacro="http://www.ros.org/wiki/xacro" >
     <joint name="camera_joint" type="fixed">
-        <parent link="body"/>
+        <parent link="camera_pre_link"/>
         <child link="camera_link"/>
         <!-- <origin xyz="0.1 0 0.37" rpy="0 0.52 0"/> -->
-        <origin xyz="0.1 0 0.2" rpy="0 0 0"/>
+        <!-- <origin xyz="0 0 0" rpy="0 0.52 0"/> -->
+        <origin xyz="0 0 0" rpy="0 0.52 -0.8"/>
     </joint>
     <link name="camera_link">
@@ -14,4 +15,18 @@
             <material name="red"/>
         </visual>
+    </link>
+    <joint name="camera_pre_joint" type="fixed">
+        <parent link="body"/>
+        <child link="camera_pre_link"/>
+        <!-- <origin xyz="0.1 0 0.37" rpy="0 0.52 0"/> -->
+        <origin xyz="0.1 0.1 0.3" rpy="0 0 0"/>
+    </joint>
+    <link name="camera_pre_link">
+        <!-- <visual>
+            <geometry>
+                <box size="0.01 0.03 0.03"/>
+            </geometry>
+            <material name="red"/>
+        </visual> -->
     </link>
     <joint name="camera_optical_joint" type="fixed">
@@ -32,10 +47,10 @@
                 <image>
                     <format>B8G8R8</format>
-                    <width>640</width>
-                    <height>420</height>
+                    <width>100</width>
+                    <height>100</height>
                 </image>
                 <clip>
-                    <near>0.05</near>
-                    <far>8</far>
+                    <near>0.15</near>
+                    <far>1.5</far>
                 </clip>
             </camera>

File: src/shesnar/urdf/robot.urdf.xacro (robot description, xacro)
@@ -3,5 +3,5 @@
     <xacro:include filename="robot_core.xacro"/>
     <xacro:include filename="lidar.xacro"/>
-    <xacro:include filename="gripper.xacro"/>
+    <!-- <xacro:include filename="gripper.xacro"/>  -->
     <xacro:include filename="depth_camera.xacro"/>
 </robot>

Commit message: setup camera detection

File: src/shesnar/urdf/depth_camera.xacro (robot description, xacro)
@@ -6,5 +6,5 @@
         <!-- <origin xyz="0.1 0 0.37" rpy="0 0.52 0"/> -->
         <!-- <origin xyz="0 0 0" rpy="0 0.52 0"/> -->
-        <origin xyz="0 0 0" rpy="0 0.52 -0.8"/>
+        <origin xyz="0 0 0" rpy="0.4 1.3 0.4"/>
     </joint>
     <link name="camera_link">
@@ -20,5 +20,5 @@
         <child link="camera_pre_link"/>
         <!-- <origin xyz="0.1 0 0.37" rpy="0 0.52 0"/> -->
-        <origin xyz="0.1 0.1 0.3" rpy="0 0 0"/>
+        <origin xyz="0.18 0.1 0.3" rpy="0 0 0"/>
     </joint>
     <link name="camera_pre_link">
@@ -51,5 +51,5 @@
                 </image>
                 <clip>
-                    <near>0.15</near>
+                    <near>0.1</near>
                     <far>1.5</far>
                 </clip>

Commit message: added second camera to robot

File: src/shesnar/urdf/depth_camera.xacro (robot description, xacro)
@@ -1,12 +1,13 @@
 <?xml version="1.0"?>
 <robot xmlns:xacro="http://www.ros.org/wiki/xacro" >
-    <joint name="camera_joint" type="fixed">
-        <parent link="camera_pre_link"/>
-        <child link="camera_link"/>
+    <!-- Left camera -->
+    <joint name="camera_joint_left" type="fixed">
+        <parent link="camera_pre_link_left"/>
+        <child link="camera_link_left"/>
         <!-- <origin xyz="0.1 0 0.37" rpy="0 0.52 0"/> -->
         <!-- <origin xyz="0 0 0" rpy="0 0.52 0"/> -->
         <origin xyz="0 0 0" rpy="0.4 1.3 0.4"/>
     </joint>
-    <link name="camera_link">
+    <link name="camera_link_left">
         <visual>
             <geometry>
@@ -16,11 +17,11 @@
         </visual>
     </link>
-    <joint name="camera_pre_joint" type="fixed">
+    <joint name="camera_pre_joint_left" type="fixed">
         <parent link="body"/>
-        <child link="camera_pre_link"/>
+        <child link="camera_pre_link_left"/>
         <!-- <origin xyz="0.1 0 0.37" rpy="0 0.52 0"/> -->
         <origin xyz="0.18 0.1 0.3" rpy="0 0 0"/>
     </joint>
-    <link name="camera_pre_link">
+    <link name="camera_pre_link_left">
         <!-- <visual>
             <geometry>
@@ -30,13 +31,13 @@
         </visual> -->
     </link>
-    <joint name="camera_optical_joint" type="fixed">
-        <parent link="camera_link"/>
-        <child link="camera_link_optical"/>
+    <joint name="camera_optical_joint_left" type="fixed">
+        <parent link="camera_link_left"/>
+        <child link="camera_link_optical_left"/>
         <origin xyz="0 0 0" rpy="-1.5708 0 -1.5708"/>
     </joint>
-    <link name="camera_link_optical"></link>
-    <gazebo reference="camera_link">
+    <link name="camera_link_optical_left"></link>
+    <gazebo reference="camera_link_left">
         <material>Gazebo/Red </material>
-        <sensor name="camera" type="depth_camera">
+        <sensor name="camera_left" type="depth_camera">
             <pose> 0 0 0 0 0 0 </pose>
             <visualize>true</visualize>
@@ -56,5 +57,64 @@
             </camera>
             <!-- <topic>camera/image_raw</topic> -->
-            <gz_frame_id>camera_link</gz_frame_id>
+            <gz_frame_id>camera_link_left</gz_frame_id>
+        </sensor>
+    </gazebo>
+    <!-- Right camera -->
+    <joint name="camera_joint_right" type="fixed">
+        <parent link="camera_pre_link_right"/>
+        <child link="camera_link_right"/>
+        <!-- <origin xyz="0.1 0 0.37" rpy="0 0.52 0"/> -->
+        <!-- <origin xyz="0 0 0" rpy="0 0.52 0"/> -->
+        <origin xyz="0 0 0" rpy="-0.4 1.3 -0.4"/>
+    </joint>
+    <link name="camera_link_right">
+        <visual>
+            <geometry>
+                <box size="0.01 0.03 0.03"/>
+            </geometry>
+            <material name="red"/>
+        </visual>
+    </link>
+    <joint name="camera_pre_joint_right" type="fixed">
+        <parent link="body"/>
+        <child link="camera_pre_link_right"/>
+        <!-- <origin xyz="0.1 0 0.37" rpy="0 0.52 0"/> -->
+        <origin xyz="0.18 -0.1 0.3" rpy="0 0 0"/>
+    </joint>
+    <link name="camera_pre_link_right">
+        <!-- <visual>
+            <geometry>
+                <box size="0.01 0.03 0.03"/>
+            </geometry>
+            <material name="red"/>
+        </visual> -->
+    </link>
+    <joint name="camera_optical_joint_right" type="fixed">
+        <parent link="camera_link_right"/>
+        <child link="camera_link_optical_right"/>
+        <origin xyz="0 0 0" rpy="-1.5708 0 -1.5708"/>
+    </joint>
+    <link name="camera_link_optical_right"></link>
+    <gazebo reference="camera_link_right">
+        <material>Gazebo/Red </material>
+        <sensor name="camera_right" type="depth_camera">
+            <pose> 0 0 0 0 0 0 </pose>
+            <visualize>true</visualize>
+            <update_rate>10</update_rate>
+            <camera>
+                <camera_info_topic>camera/camera_info</camera_info_topic>
+                <horizontal_fow>1.089</horizontal_fow>
+                <image>
+                    <format>B8G8R8</format>
+                    <width>100</width>
+                    <height>100</height>
+                </image>
+                <clip>
+                    <near>0.1</near>
+                    <far>1.5</far>
+                </clip>
+            </camera>
+            <!-- <topic>camera/image_raw</topic> -->
+            <gz_frame_id>camera_link_right</gz_frame_id>
         </sensor>
     </gazebo>
