Commit message: move to docker

File: src/shesnar/urdf/lidar.xacro (robot description, xacro)
@@ -22,9 +22,9 @@
     </link>
     <gazebo reference="laser_frame">
-        <sensor name="laser" type="ray">
+        <sensor name="laser" type="gpu_lidar">
             <pose> 0 0 0 0 0 0 </pose>
             <visualize>true</visualize>
             <update_rate>10</update_rate>
-            <ray>
+            <lidar>
                 <scan>
                     <horizontal>
@@ -38,12 +38,7 @@
                     <max>12</max>
                 </range>
-            </ray>
-            <plugin name="laser_controller" filename="libgazebo_ros_ray_sensor.so">
-                <ros>
-                    <argument>~/out:=scan</argument>
-                </ros>
-                <output_type>sensor_msgs/LaserScan</output_type>
-                <frame_name>laser_frame</frame_name>
-            </plugin>
+            </lidar>
+            <topic>scan</topic>
+            <gz_frame_id>laser_frame</gz_frame_id>
         </sensor>
     </gazebo>

File: src/shesnar/urdf/robot_core.xacro (robot description, xacro)
@@ -25,5 +25,5 @@
             <origin xyz="0.1 -0.18 0" rpy="0 0 1.57" />
             <geometry>
-                <mesh filename="package://shesnar/meshes/body.dae" scale="0.001 0.001 0.001" rpy="0 0 1.04"/>
+                <mesh scale="0.001 0.001 0.001" rpy="0 0 1.04" filename="file://$(find shesnar)/meshes/body.obj"/>
             <!-- <cylinder radius="0.20" length="0.12"/> -->
             </geometry>
@@ -42,3 +42,16 @@
         </xacro:inertial_cylinder>
     </link>
+      <!-- <gazebo> -->
+        <!-- <plugin name="gz::sim::systems::OdometryPublisher" filename="gz-sim-odometry-publisher-system">
+            <odom_frame>odom</odom_frame>
+            <robot_base_frame>base_link</robot_base_frame>
+            <odom_publish_frequency>50</odom_publish_frequency>
+            <odom_topic>/odom</odom_topic>
+            <tf_topic>/tf</tf_topic>
+        </plugin> -->
+<!--
+        <plugin name="gz::sim::systems::VelocityControl" filename="gz-sim-velocity-control-system">
+            <topic>/cmd_vel</topic>
+        </plugin> -->
+    <!-- </gazebo> -->
 </robot>

Commit message: cus & mayaks setup

File: src/shesnar/urdf/lidar.xacro (robot description, xacro)
@@ -4,5 +4,5 @@
         <parent link="body"/>
         <child link="laser_frame"/>
-        <origin xyz="0 0 0.18" rpy="0 0 -2.085"/>
+        <origin xyz="0 0 0.41" rpy="0 0 -2.085"/>
     </joint>
     <link name="laser_frame">

Commit message: aruco fix

File: src/shesnar/urdf/lidar.xacro (robot description, xacro)
@@ -43,3 +43,20 @@
         </xacro:inertial_cylinder>
     </link>
+    <link name="aruco">
+        <visual>
+            <geometry>
+                <box size="0.1 0.1 0.005"/>
+            </geometry>
+        </visual>
+        <collision>
+            <geometry>
+                <box size="0.1 0.1 0.005"/>
+            </geometry>
+        </collision>
+    </link>
+    <joint name="aruco_joint" type="fixed">
+        <parent link="laser_frame"/>
+        <child link="aruco"/>
+        <origin xyz="0 0 0.0225" rpy="0 0 2.085"/>
+    </joint>
 </robot>

Commit message: visual_odom beta

File: src/shesnar/urdf/lidar.xacro (robot description, xacro)
@@ -46,17 +46,12 @@
         <visual>
             <geometry>
-                <box size="0.1 0.1 0.005"/>
+                 <mesh filename="/eurobot_2025/src/shesnar/meshes/aruco_plane.obj" scale="0.5 0.5 0.5"/>
             </geometry>
         </visual>
-        <collision>
-            <geometry>
-                <box size="0.1 0.1 0.005"/>
-            </geometry>
-        </collision>
     </link>
     <joint name="aruco_joint" type="fixed">
         <parent link="laser_frame"/>
         <child link="aruco"/>
-        <origin xyz="0 0 0.0225" rpy="0 0 2.085"/>
+        <origin xyz="0 0 0.0225" rpy="1.571 0 2.085"/>
     </joint>
 </robot>

Commit message: micro fix

File: src/shesnar/urdf/lidar.xacro (robot description, xacro)
@@ -46,5 +46,5 @@
         <visual>
             <geometry>
-                 <mesh filename="/eurobot_2025/src/shesnar/meshes/aruco_plane.obj" scale="0.5 0.5 0.5"/>
+                 <mesh filename="file://$(find shesnar)/meshes/aruco_plane.obj" scale="0.5 0.5 0.5"/>
             </geometry>
         </visual>

Commit message: update

File: src/shesnar/urdf/lidar.xacro (robot description, xacro)
@@ -26,5 +26,5 @@
         <parent link="body"/>
         <child link="laser_frame"/>
-        <origin xyz="0 0 0.41" rpy="0 0 -2.085"/>
+        <origin xyz="0 0 0.41" rpy="0 3.14 0"/>
     </joint>
     <link name="laser_frame">
